File: boards/pmod-mmcx/pmod-mmcx.kicad_pcb (KiCad board)
At the start: 4 copper layers, 59 x 20 mm, 13 parts, among them J1 PMOD_DEVICE_DIFF, P1 MMCX, P2 MMCX, P3 MMCX, P4 MMCX, P5 MMCX, P6 MMCX, P7 MMCX, P8 MMCX, P9 MMCX

Commit message: Changed mask clearance
Other:
- rule pad_to_mask_clearance: 0.2 -> 0.05
Changed lines of the file:
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@@
 (kicad_pcb (version 20170123) (host pcbnew "(2017-05-24 revision 38c8470)-master")
   (general
-    (links 0)
+    (links 47)
     (no_connects 0)
     (area 37.4625 25.969285 100.403572 48.100001)
@@
     (pad_size 1.524 1.524)
     (pad_drill 0.762)
-    (pad_to_mask_clearance 0.2)
+    (pad_to_mask_clearance 0.05)
     (aux_axis_origin 0 0)
     (visible_elements FFFFFF7F)
