File: boards/resistive-probe/resistive-probe.kicad_pcb (KiCad board)
At the start: 2 copper layers, 60.5 x 9 mm, 14 parts, among them P1 MMCX, P2 SOLDERPAD, P3 SOLDERPAD

Commit message: Updated resistive probe to be more manufacturable
Parts:
- removed the G*** at (91.0, 50.5)
- moved G*** 48.8 mm to (93.2, 50.5), turned to 270 degrees
Other:
- board size 60.5 x 9 mm -> 60.5 x 6 mm
- board text added: "STARSHIPRAIDER Probe / A. Zonenberg / v0.2 / 2017-11-30"
- board text removed: "A. Zonenberg / 2017-05-27"
- board text removed: "STARSHIPRAIDER Resistive Probe v0.1"
