File: boards/sma-probetarget/sma-probetarget.kicad_pcb (KiCad board)
At the start: 4 copper layers, 59 x 23 mm, 10 parts, among them J1 Conn_Coaxial, J2 Conn_Coaxial, J3 Conn_Coaxial, J4 Conn_Coaxial, J5 Conn_01x01, J6 Conn_01x01, J7 Conn_01x01

Commit message: Updated zone fills
Routing:
- added copper zone on In1.Cu, net /GND
- removed copper zone on In1.Cu, net (none)
Changed lines of the file:
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@@
     (user_trace_width 0.41)
     (trace_clearance 0.1)
-    (zone_clearance 0.508)
+    (zone_clearance 0.2)
     (zone_45_only no)
     (trace_min 0.2)
@@
   (segment (start 62.1 55) (end 116.9 55) (width 0.41) (layer F.Cu) (net 2))
   (segment (start 62.1 68) (end 116.9 68) (width 0.41) (layer F.Cu) (net 3))
-  (zone (net 0) (net_name "") (layer In1.Cu) (hatch edge 0.508)
+  (zone (net 1) (net_name /GND) (layer In1.Cu) (hatch edge 0.508)
     (connect_pads (clearance 0.2))
     (min_thickness 0.1)
