File: boards/diffprobe-calibrated-prototype/sigpath.sch (KiCad schematic (older format))
At the start: 14 parts

Commit message: Continued work on differential probe
Parts:
- added C? (x2): 4.7 uF, symbol C
- added C? (x4): 0.47 uF, symbol C
- added C? (x2): 0.1 uF, symbol C
- added C? (x4): 0.1 uF 25V, symbol C
- added K? (x2): AXICOM_HF3_2COIL, symbol AXICOM_HF3_2COIL
- added R? (x3): 0, symbol R
- added R? (x2): 2, symbol R
- added U?: AD5752, symbol AD57x2
- added U?: MCP1501_DFN, symbol MCP1501_DFN
- added U? (x2): DRV8800_WQFN, symbol DRV8800_WQFN
Connections:
- net labels added: 12V0_P, 2V5_REF, 3V3, COIL1_N, COIL1_P, COIL2_N, COIL2_P, HBRIDGE_MODE, RELAY1_DIR, RELAY1_EN, RELAY2_DIR, RELAY2_EN, SPI_CS_N, SPI_MISO, SPI_MOSI, SPI_SCK, VIN_N_AC, VIN_N_COUPLED, VIN_P_AC, VIN_P_COUPLED
- wire segments 49 -> 168
- no-connect marks 5 -> 9
Other:
- note added: "2R = overcurrent @ 250 mA"
- note added: "TODO: Diodes on relay coils"
- note added: "TODO: snubber diode etc"
- note added: "VOUT should not exceed 5V RMS to avoid damaging DSO\nVOUT_RAW should not exceed +18 dBm (1.776 Vrms / 5V p-p) AC voltage\nHMC346AMS doesn't specify max DC offset other than "should be about zero"\nWith 2V/V gain:\n* Input differential = 0.89 Vrms max (17.76V w/ 20x probes)\n* Input common mode = unspecified, but minimize"
- note removed: "VOUT should not exceed 5V RMS to avoid damaging DSO\nVOUT_RAW should not exceed +18 dBm (1.776 Vrms / 5V p-p) AC voltage\nHMC346AMS doesn't specify max common mode voltage other than "should be about zero"\nWith 2V/V gain:\n* Input differential = 0.89 Vrms max (17.76V w/ 20x probes)\n* Input common mode = unspecified"
- moved on the sheet: D?, P?, R?, U?

Commit message: Finished adding decoupling caps etc. Still needs signoff review.
Parts:
- added C22, C29: 22 uF 25V, symbol C
- added C23, C25, C26, C32, C35: 4.7 uF, symbol C
- added C24, C27, C28, C30, C34, C36: 0.47 uF, symbol C
- added C31, C33: 0.1 uF 25V, symbol C
- added R18, R19, R20, R21: 0, symbol R
- gave numbers to parts that had none: 37
Connections:
- net 12V0_P: now also C22.1, C29.1, C31.1, C33.1
- net 3V3: now also C23.1, C24.1, C30.1, R18.2, R19.2, R20.2, R21.2; no longer U2.3 (SLEEP_N), U3.3 (SLEEP_N)
- net 5V0_N: now also C26.2, C28.2, C35.1, C36.1
- net 5V0_P: now also C25.1, C27.1, C32.1, C34.1
- net COIL1_P: no longer U3.9 (OUT_N)
- net COIL2_P: now also U3.9 (OUT_N)
- net GND: now also R1.2, R2.1, C22.2, C23.2, C24.2, C25.2, C26.1, C27.2, C28.1, C29.2, C30.2, C31.2, C32.2, C33.2, C34.2, C35.2, C36.2; no longer R1.1, R2.2
- net VIN_N: no longer R2.1
- net VIN_N_COUPLED: now also R1.1
- net VIN_P: no longer R1.2
- net VIN_P_COUPLED: now also R2.2
- net HBRIDGE_MODE: no longer names the net of U2.16 (MODE)
- net HBRIDGE_MODE: now also R18.1; no longer U3.16 (MODE)
- new net: R19.1, U2.3 (SLEEP_N)
- new net: R20.1, U3.16 (MODE)
- new net: R21.1, U3.3 (SLEEP_N)
Other:
- note added: "Attenuator FB amp decoupling"
- note added: "DAC decoupling"
- note added: "Diff amp decoupling"
- note added: "H-bridge decoupling"
- note added: "VREF decoupling"
- note removed: "TODO: Decoupling for everything"
- note removed: "TODO: Diodes on relay coils"
- note removed: "TODO: snubber diode etc"
- moved on the sheet: C1, C10, C11, C12, C2, C3, C4, C5, C6, C7, C8, C9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

Commit message: Finished initial schematic review
Parts:
- added C43, C45: 4.7 uF, symbol C
- added C44, C46: 0.47 uF, symbol C
- added TP1, TP2, TP3: CONN_01X01, symbol CONN_01X01
Connections:
- net 12V0_P: now also U2.8 (VBB), U3.8 (VBB); no longer U2.2 (GND), U3.2 (GND)
- net ATTEN_REF: now also U7.4 (I)
- net ATTEN_V2: now also U7.3 (V2)
- net COIL1_N: now also U2.9 (OUT_N)
- net COIL1_P: now also U2.6 (OUT_P); no longer U2.9 (OUT_N)
- net COIL2_N: now also U3.9 (OUT_N)
- net COIL2_P: now also U3.6 (OUT_P); no longer U3.9 (OUT_N)
- net GND: now also U2.2 (GND), U3.2 (GND), U7.2 (GND), C43.2, C44.2, C45.2, C46.2
- net VATTEN: now also U7.6 (V1), C43.1, C44.1, TP1.1 (P1); no longer U7.3 (V2)
- net VATTEN_P: now also TP2.1 (P1)
- net VOFFSET: now also C45.1, C46.1, TP3.1 (P1)
- net VOUT: now also U7.8 (RF2)
- net VOUT_RAW: now also U7.1 (RF1); no longer U7.4 (I)
Other:
- note added: "Capacitive filtering to reduce noise on DAC outputs"
- moved on the sheet: U7
Changed lines of the file:
@@
 Sheet 2 4
 Title "500 MHz Active Differential Probe"
-Date "2017-12-19"
+Date "2017-12-20"
 Rev "0.2"
 Comp "Andrew D. Zonenberg"
@@
 Text Label 1050 1500 2    60   ~ 0
 GND
-Wire Wire Line
-	5450 6100 5450 6150
-Wire Wire Line
-	5450 6150 5700 6150
-Wire Wire Line
-	5450 6300 5450 6250
-Wire Wire Line
-	5450 6250 5700 6250
 Text Label 1500 1800 0    60   ~ 0
 VIN_P
@@
 L HMC346AMS8GE U7
 U 1 1 5A1FD030
-P 10150 6850
-F 0 "U7" H 10425 7797 60  0000 C CNN
-F 1 "HMC346AMS8GE" H 10425 7691 60  0000 C CNN
-F 2 "" H 10350 6850 60  0001 C CNN
-F 3 "" H 10350 6850 60  0001 C CNN
-	1    10150 6850
+P 10150 6950
+F 0 "U7" H 10200 7950 60  0000 C CNN
+F 1 "HMC346AMS8GE" H 10500 7850 60  0000 C CNN
+F 2 "" H 10350 6950 60  0001 C CNN
+F 3 "" H 10350 6950 60  0001 C CNN
+	1    10150 6950
 	1    0    0    -1
 $EndComp
@@
 	9800 6700 9950 6700
 Wire Wire Line
-	9850 6700 9850 6800
+	9850 6700 9850 6900
 Wire Wire Line
 	9850 6800 9950 6800
@@
 	-1   0    0    -1
 $EndComp
-Text Label 5450 6100 2    60   ~ 0
+Text Label 5600 6150 2    60   ~ 0
 VIN_P_COUPLED
-Text Label 5450 6300 2    60   ~ 0
+Text Label 5600 6250 2    60   ~ 0
 VIN_N_COUPLED
 $Comp
@@
 Text Label 4000 3400 0    60   ~ 0
 COIL2_N
-Text HLabel 6150 900  0    60   Input ~ 0
+Text HLabel 6150 800  0    60   Input ~ 0
 12V0_P
 Text HLabel 6400 1700 0    60   Input ~ 0
@@
 U 1 1 5A377542
 P 6700 1750
-F 0 "U2" H 7125 2847 60  0000 C CNN
-F 1 "DRV8800_WQFN" H 7125 2741 60  0000 C CNN
+F 0 "U2" H 6750 2800 60  0000 C CNN
+F 1 "DRV8800_WQFN" H 7050 1700 60  0000 C CNN
 F 2 "" H 6700 1750 60  0001 C CNN
 F 3 "" H 6700 1750 60  0001 C CNN
@@
 	6500 1000 6400 1000
 Wire Wire Line
-	6400 1000 6400 1100
+	6400 900  6400 1100
 Wire Wire Line
 	6400 1100 6500 1100
@@
 GND
 Wire Wire Line
-	6150 900  6500 900
+	6150 800  6500 800
 NoConn ~ 6500 1200
 Wire Wire Line
@@
 Wire Wire Line
 	8450 1700 8450 1800
+Text Label 7850 800  0    60   ~ 0
+COIL1_P
+Wire Wire Line
+	7850 800  7750 800
 Text Label 7850 900  0    60   ~ 0
-COIL1_P
+COIL1_N
 Wire Wire Line
 	7850 900  7750 900
-Text Label 7850 1000 0    60   ~ 0
-COIL1_N
-Wire Wire Line
-	7850 1000 7750 1000
 NoConn ~ 7750 1600
 Wire Wire Line
@@
 U 1 1 5A37A03C
 P 6700 3300
-F 0 "U3" H 7125 4397 60  0000 C CNN
-F 1 "DRV8800_WQFN" H 7125 4291 60  0000 C CNN
+F 0 "U3" H 6750 4350 60  0000 C CNN
+F 1 "DRV8800_WQFN" H 7050 3250 60  0000 C CNN
 F 2 "" H 6700 3300 60  0001 C CNN
 F 3 "" H 6700 3300 60  0001 C CNN
@@
 	6500 2550 6400 2550
 Wire Wire Line
-	6400 2550 6400 2650
+	6400 2450 6400 2650
 Wire Wire Line
 	6400 2650 6500 2650
@@
 GND
 Wire Wire Line
-	6150 2450 6500 2450
+	6150 2350 6500 2350
 NoConn ~ 6500 2750
 Wire Wire Line
@@
 Wire Wire Line
 	8450 3250 8450 3350
+Text Label 7850 2350 0    60   ~ 0
+COIL2_P
+Wire Wire Line
+	7850 2350 7750 2350
 Text Label 7850 2450 0    60   ~ 0
-COIL2_P
+COIL2_N
 Wire Wire Line
 	7850 2450 7750 2450
-Text Label 7850 2550 0    60   ~ 0
-COIL2_N
-Wire Wire Line
-	7850 2550 7750 2550
 NoConn ~ 7750 3150
 Wire Wire Line
@@
 Text Notes 7750 3650 0    60   ~ 0
 2R = overcurrent @ 250 mA
-Text Label 6150 2450 2    60   ~ 0
+Text Label 6150 2350 2    60   ~ 0
 12V0_P
 Wire Wire Line
@@
 	1200 9650 1850 9650
 Connection ~ 1350 9650
+Wire Wire Line
+	6400 900  6500 900
+Connection ~ 6400 1000
+Wire Wire Line
+	6400 2450 6500 2450
+Connection ~ 6400 2550
+Text Notes 5400 9550 0    60   ~ 0
+Capacitive filtering to reduce noise on DAC outputs
+$Comp
+L C C44
+U 1 1 5A3B3EBD
+P 6000 9250
+F 0 "C44" H 6115 9296 50  0000 L CNN
+F 1 "0.47 uF" H 6115 9205 50  0000 L CNN
+F 2 "" H 6038 9100 50  0000 C CNN
+F 3 "" H 6000 9250 50  0000 C CNN
+	1    6000 9250
+	1    0    0    -1
+$EndComp
+$Comp
+L C C43
+U 1 1 5A3B3FBD
+P 5500 9250
+F 0 "C43" H 5615 9296 50  0000 L CNN
+F 1 "4.7 uF" H 5615 9205 50  0000 L CNN
+F 2 "" H 5538 9100 50  0000 C CNN
+F 3 "" H 5500 9250 50  0000 C CNN
+	1    5500 9250
+	1    0    0    -1
+$EndComp
+Text Label 5350 9100 2    60   ~ 0
+VATTEN
+Wire Wire Line
+	5350 9100 6000 9100
+Connection ~ 5500 9100
+Text Label 5350 9400 2    60   ~ 0
+GND
+Wire Wire Line
+	5350 9400 6000 9400
+Connection ~ 5500 9400
+$Comp
+L C C46
+U 1 1 5A3B4ABF
+P 7500 9250
+F 0 "C46" H 7615 9296 50  0000 L CNN
+F 1 "0.47 uF" H 7615 9205 50  0000 L CNN
+F 2 "" H 7538 9100 50  0000 C CNN
+F 3 "" H 7500 9250 50  0000 C CNN
+	1    7500 9250
+	1    0    0    -1
+$EndComp
+$Comp
+L C C45
+U 1 1 5A3B4AC5
+P 7000 9250
+F 0 "C45" H 7115 9296 50  0000 L CNN
+F 1 "4.7 uF" H 7115 9205 50  0000 L CNN
+F 2 "" H 7038 9100 50  0000 C CNN
+F 3 "" H 7000 9250 50  0000 C CNN
+	1    7000 9250
+	1    0    0    -1
+$EndComp
+Text Label 6850 9100 2    60   ~ 0
+VOFFSET
+Wire Wire Line
+	6850 9100 7500 9100
+Connection ~ 7000 9100
+Text Label 6850 9400 2    60   ~ 0
+GND
+Wire Wire Line
+	6850 9400 7500 9400
+Connection ~ 7000 9400
+Wire Wire Line
+	9850 6900 9950 6900
+Connection ~ 9850 6800
+Wire Wire Line
+	5600 6150 5700 6150
+Wire Wire Line
+	5700 6250 5600 6250
+$Comp
+L CONN_01X01 TP1
+U 1 1 5A3B854B
+P 11600 3300
+F 0 "TP1" H 11678 3341 50  0000 L CNN
+F 1 "CONN_01X01" H 11678 3250 50  0000 L CNN
+F 2 "" H 11600 3300 50  0000 C CNN
+F 3 "" H 11600 3300 50  0000 C CNN
+	1    11600 3300
+	1    0    0    -1
+$EndComp
+Text Label 11400 3300 2    60   ~ 0
+VATTEN
+$Comp
+L CONN_01X01 TP2
+U 1 1 5A3B8754
+P 11600 3600
+F 0 "TP2" H 11678 3641 50  0000 L CNN
+F 1 "CONN_01X01" H 11678 3550 50  0000 L CNN
+F 2 "" H 11600 3600 50  0000 C CNN
+F 3 "" H 11600 3600 50  0000 C CNN
+	1    11600 3600
+	1    0    0    -1
+$EndComp
+Text Label 11400 3600 2    60   ~ 0
+VATTEN_P
+$Comp
+L CONN_01X01 TP3
+U 1 1 5A3B8866
+P 11600 3900
+F 0 "TP3" H 11678 3941 50  0000 L CNN
+F 1 "CONN_01X01" H 11678 3850 50  0000 L CNN
+F 2 "" H 11600 3900 50  0000 C CNN
+F 3 "" H 11600 3900 50  0000 C CNN
+	1    11600 3900
+	1    0    0    -1
+$EndComp
+Text Label 11400 3900 2    60   ~ 0
+VOFFSET
 $EndSCHEMATC

Commit message: Initial layout
Parts:
- C1, C2, C23, C25, C26, C32, C35, C43, C45: footprint (none) -> azonenberg_pcb:EIA_0603_CAP_NOSILK
- C10, C11, C12, C24, C27, C28, C3, C30, C31, C33, C34, C36, C4, C44, C46, C5, C6, C7, C8, C9: footprint (none) -> azonenberg_pcb:EIA_0402_CAP_NOSILK
- C22, C29: footprint (none) -> azonenberg_pcb:EIA_1812_CAP_NOSILK
- D1: footprint (none) -> azonenberg_pcb:SOD123
- J4, J5, J6: footprint (none) -> azonenberg_pcb:CONN_SMA_EDGE_SAMTEC_SMA_J_P_H_ST_EM1
- K1, K2: footprint (none) -> azonenberg_pcb:RELAY_TE_HF3_2COIL_50OHM
- R1, R10, R11, R12, R18, R19, R2, R20, R21, R3, R4, R5, R6, R7, R8, R9: footprint (none) -> azonenberg_pcb:EIA_0402_RES_NOSILK
- TP1, TP2, TP3: footprint (none) -> azonenberg_pcb:TESTPOINT_SMT_0.5MM
- U1: footprint (none) -> azonenberg_pcb:DFN_8_0.5MM_2x2MM
- U2, U3, U5: footprint (none) -> azonenberg_pcb:QFN_16_0.65MM_4x4MM
- U4: footprint (none) -> azonenberg_pcb:TSSOP_24_0.65MM_5MM_EPAD_5x3p2
- U6: footprint (none) -> azonenberg_pcb:SOP_8_0.5MM_3MM
- U7: footprint (none) -> azonenberg_pcb:SOP_8_0.5MM_3MM_EPAD

Commit message: Moved a bunch of old files out of the way, added some notes that never got committed
Parts:
- C1, C10, C11, C12, C2, C22, C23, C24, C25, C26, C27, C28, C29, C3, C30, C31, C32, C33, C34, C35, C36, C4, C43, C44, C45, C46, C5, C6, C7, C8, C9: symbol C -> device:C
- D1: symbol D -> device:D
- J4, J5, J6: symbol BNC -> diffprobe-calibrated-prototype-rescue:BNC
- K1, K2: symbol AXICOM_HF3_2COIL -> special-azonenberg:AXICOM_HF3_2COIL
- R1, R10, R11, R12, R18, R19, R2, R20, R21, R3, R4, R5, R6, R7, R8, R9: symbol R -> device:R
- TP1, TP2, TP3: symbol CONN_01X01 -> diffprobe-calibrated-prototype-rescue:CONN_01X01
- U1: symbol MCP1501_DFN -> analog-azonenberg:MCP1501_DFN
- U2, U3: symbol DRV8800_WQFN -> special-azonenberg:DRV8800_WQFN
- U4: symbol AD57x2 -> analog-azonenberg:AD57x2
- U5: symbol THS3217 -> analog-azonenberg:THS3217
- U6: symbol AD8675 -> analog-azonenberg:AD8675
- U7: symbol HMC346AMS8GE -> analog-azonenberg:HMC346AMS8GE
