File: boards/entry-afe-characterization/psu.sch (KiCad schematic (older format))
At the start: 79 parts, among them J10 CONN_3_PWROUT, Q2 2SA2039-TL-E, U10 LT3042, U11 LT3042, U12 MCP1501T-25E/RW, U13 LT3093, U14 PTN78000AAZ, U15 LT3093, U16 LT3042, U17 TL431ACDBZR, U8 TPS54227-DRC, U9 LT3042

Commit message: Continued assigning footprints
Parts:
- L4: footprint (none) -> azonenberg_pcb:INDUCTOR_YUDEN_NR6028
- Q2: footprint (none) -> azonenberg_pcb:TO_253
- R11, R38, R42, R44, R46, R51, R58: footprint (none) -> azonenberg_pcb:EIA_0402_RES_NOSILK
- R39: value 180.1K -> 180K; footprint (none) -> azonenberg_pcb:EIA_0402_RES_NOSILK
- R40, R52: value 470 -> 470 1%; footprint (none) -> azonenberg_pcb:EIA_0402_RES_NOSILK
- R41: value 4.7K -> 4.7K 1%; footprint (none) -> azonenberg_pcb:EIA_0402_RES_NOSILK
- R43, R56: value 60K 1% -> 60.4K 1%; footprint (none) -> azonenberg_pcb:EIA_0402_RES_NOSILK
- R45: value 2.7K -> 2.7K 1%; footprint (none) -> azonenberg_pcb:EIA_0402_RES_NOSILK
- R47: value 6.4K -> 6.49K 1%; footprint (none) -> azonenberg_pcb:EIA_0402_RES_NOSILK
- R48: value 3.6K -> 3.6K 1%; footprint (none) -> azonenberg_pcb:EIA_0402_RES_NOSILK
- R49: value 8.0K -> 8.06K 1%; footprint (none) -> azonenberg_pcb:EIA_0402_RES_NOSILK
- R50: value 2.0K -> 2K 1%; footprint (none) -> azonenberg_pcb:EIA_0402_RES_NOSILK
- R54: value 9.0K -> 9.09K 1%; footprint (none) -> azonenberg_pcb:EIA_0402_RES_NOSILK
- R55: value 1.0K -> 1K 1%; footprint (none) -> azonenberg_pcb:EIA_0402_RES_NOSILK
- R57: value 60K 1% -> 49.9K 1%; footprint (none) -> azonenberg_pcb:EIA_0402_RES_NOSILK
Changed lines of the file:
@@
 F 0 "L4" V 2792 1700 40  0000 C CNN
 F 1 "4.7 uH" V 2868 1700 40  0000 C CNN
-F 2 "" H 2950 1700 60  0001 C CNN
+F 2 "azonenberg_pcb:INDUCTOR_YUDEN_NR6028" H 2950 1700 60  0001 C CNN
 F 3 "" H 2950 1700 60  0000 C CNN
 	1    2950 1700
@@
 F 0 "R11" V 1200 2300 50  0000 C CNN
 F 1 "10K" V 1300 2300 50  0000 C CNN
-F 2 "" V 1230 2300 50  0001 C CNN
+F 2 "azonenberg_pcb:EIA_0402_RES_NOSILK" V 1230 2300 50  0001 C CNN
 F 3 "" H 1300 2300 50  0001 C CNN
 	1    1300 2300
@@
 F 0 "R38" H 3650 2300 50  0000 C CNN
 F 1 "22.1K" H 3800 2600 50  0000 C CNN
-F 2 "" V 3730 2350 50  0001 C CNN
+F 2 "azonenberg_pcb:EIA_0402_RES_NOSILK" V 3730 2350 50  0001 C CNN
 F 3 "" H 3800 2350 50  0001 C CNN
 	1    3800 2350
@@
 P 3050 2350
 F 0 "R39" H 2900 2300 50  0000 C CNN
-F 1 "180.1K" H 3050 2600 50  0000 C CNN
-F 2 "" V 2980 2350 50  0001 C CNN
+F 1 "180K" H 3050 2600 50  0000 C CNN
+F 2 "azonenberg_pcb:EIA_0402_RES_NOSILK" V 2980 2350 50  0001 C CNN
 F 3 "" H 3050 2350 50  0001 C CNN
 	1    3050 2350
@@
 F 0 "R44" V 2800 2050 50  0000 C CNN
 F 1 "0" V 2900 2050 50  0000 C CNN
-F 2 "" V 2830 2050 50  0001 C CNN
+F 2 "azonenberg_pcb:EIA_0402_RES_NOSILK" V 2830 2050 50  0001 C CNN
 F 3 "" H 2900 2050 50  0001 C CNN
 	1    2900 2050
@@
 F 0 "R42" H 3000 3950 50  0000 C CNN
 F 1 "49.9K 1%" H 3100 4150 50  0000 C CNN
-F 2 "" V 3030 3950 50  0001 C CNN
+F 2 "azonenberg_pcb:EIA_0402_RES_NOSILK" V 3030 3950 50  0001 C CNN
 F 3 "" H 3100 3950 50  0001 C CNN
 	1    3100 3950
@@
 P 3100 6200
 F 0 "R43" H 3000 6200 50  0000 C CNN
-F 1 "60K 1%" H 3100 6400 50  0000 C CNN
-F 2 "" V 3030 6200 50  0001 C CNN
+F 1 "60.4K 1%" H 3100 6400 50  0000 C CNN
+F 2 "azonenberg_pcb:EIA_0402_RES_NOSILK" V 3030 6200 50  0001 C CNN
 F 3 "" H 3100 6200 50  0001 C CNN
 	1    3100 6200
@@
 F 0 "R46" H 3000 7300 50  0000 C CNN
 F 1 "33K 1%" H 3100 7500 50  0000 C CNN
-F 2 "" V 3030 7300 50  0001 C CNN
+F 2 "azonenberg_pcb:EIA_0402_RES_NOSILK" V 3030 7300 50  0001 C CNN
 F 3 "" H 3100 7300 50  0001 C CNN
 	1    3100 7300
@@
 P 5600 6800
 F 0 "R47" V 5700 6800 50  0000 C CNN
-F 1 "6.4K " V 5600 6800 50  0000 C CNN
-F 2 "" V 5530 6800 50  0001 C CNN
+F 1 "6.49K 1%" V 5500 6750 50  0000 C CNN
+F 2 "azonenberg_pcb:EIA_0402_RES_NOSILK" V 5530 6800 50  0001 C CNN
 F 3 "" H 5600 6800 50  0001 C CNN
 	1    5600 6800
@@
 P 6050 6800
 F 0 "R48" V 6150 6800 50  0000 C CNN
-F 1 "3.6K" V 6050 6800 50  0000 C CNN
-F 2 "" V 5980 6800 50  0001 C CNN
+F 1 "3.6K 1%" V 5950 6450 50  0000 C CNN
+F 2 "azonenberg_pcb:EIA_0402_RES_NOSILK" V 5980 6800 50  0001 C CNN
 F 3 "" H 6050 6800 50  0001 C CNN
 	1    6050 6800
@@
 P 5600 7150
 F 0 "R49" V 5700 7150 50  0000 C CNN
-F 1 "8.0K" V 5600 7150 50  0000 C CNN
-F 2 "" V 5530 7150 50  0001 C CNN
+F 1 "8.06K 1%" V 5500 7150 50  0000 C CNN
+F 2 "azonenberg_pcb:EIA_0402_RES_NOSILK" V 5530 7150 50  0001 C CNN
 F 3 "" H 5600 7150 50  0001 C CNN
 	1    5600 7150
@@
 P 6050 7150
 F 0 "R50" V 6150 7150 50  0000 C CNN
-F 1 "2.0K" V 6050 7150 50  0000 C CNN
-F 2 "" V 5980 7150 50  0001 C CNN
+F 1 "2K 1%" V 6000 6850 50  0000 C CNN
+F 2 "azonenberg_pcb:EIA_0402_RES_NOSILK" V 5980 7150 50  0001 C CNN
 F 3 "" H 6050 7150 50  0001 C CNN
 	1    6050 7150
@@
 F 0 "R51" H 7620 1996 50  0000 L CNN
 F 1 "11.5K 1%" H 7620 1905 50  0000 L CNN
-F 2 "" V 7480 1950 50  0001 C CNN
+F 2 "azonenberg_pcb:EIA_0402_RES_NOSILK" V 7480 1950 50  0001 C CNN
 F 3 "" H 7550 1950 50  0001 C CNN
 	1    7550 1950
@@
 P 6600 4050
 F 0 "R56" H 6500 4050 50  0000 C CNN
-F 1 "60K 1%" H 6600 3850 50  0000 C CNN
-F 2 "" V 6530 4050 50  0001 C CNN
+F 1 "60.4K 1%" H 6600 3850 50  0000 C CNN
+F 2 "azonenberg_pcb:EIA_0402_RES_NOSILK" V 6530 4050 50  0001 C CNN
 F 3 "" H 6600 4050 50  0001 C CNN
 	1    6600 4050
@@
 Text Label 6250 5050 0    50   ~ 0
 7V0_N_2
-$Comp
-L device:R R57
-U 1 1 5E8EA1D4
-P 6600 5300
-F 0 "R57" H 6500 5300 50  0000 C CNN
-F 1 "60K 1%" H 6600 5100 50  0000 C CNN
-F 2 "" V 6530 5300 50  0001 C CNN
-F 3 "" H 6600 5300 50  0001 C CNN
-	1    6600 5300
-	1    0    0    -1
-$EndComp
 Wire Wire Line
 	6600 5150 6250 5150
@@
 P 5600 7500
 F 0 "R54" V 5700 7500 50  0000 C CNN
-F 1 "9.0K" V 5600 7500 50  0000 C CNN
-F 2 "" V 5530 7500 50  0001 C CNN
+F 1 "9.09K 1%" V 5500 7500 50  0000 C CNN
+F 2 "azonenberg_pcb:EIA_0402_RES_NOSILK" V 5530 7500 50  0001 C CNN
 F 3 "" H 5600 7500 50  0001 C CNN
 	1    5600 7500
@@
 P 6050 7500
 F 0 "R55" V 6150 7500 50  0000 C CNN
-F 1 "1.0K" V 6050 7500 50  0000 C CNN
-F 2 "" V 5980 7500 50  0001 C CNN
+F 1 "1K 1%" V 6000 7250 50  0000 C CNN
+F 2 "azonenberg_pcb:EIA_0402_RES_NOSILK" V 5980 7500 50  0001 C CNN
 F 3 "" H 6050 7500 50  0001 C CNN
 	1    6050 7500
@@
 P 8000 3450
 F 0 "R40" H 7850 3450 50  0000 C CNN
-F 1 "470" H 8150 3450 50  0000 C CNN
-F 2 "" V 7930 3450 50  0001 C CNN
+F 1 "470 1%" H 8200 3450 50  0000 C CNN
+F 2 "azonenberg_pcb:EIA_0402_RES_NOSILK" V 7930 3450 50  0001 C CNN
 F 3 "" H 8000 3450 50  0001 C CNN
 	1    8000 3450
@@
 P 8000 3900
 F 0 "R41" H 7850 3900 50  0000 C CNN
-F 1 "4.7K" H 8150 3900 50  0000 C CNN
-F 2 "" V 7930 3900 50  0001 C CNN
+F 1 "4.7K 1%" H 8200 3900 50  0000 C CNN
+F 2 "azonenberg_pcb:EIA_0402_RES_NOSILK" V 7930 3900 50  0001 C CNN
 F 3 "" H 8000 3900 50  0001 C CNN
 	1    8000 3900
@@
 P 8000 4850
 F 0 "R45" H 7850 4850 50  0000 C CNN
-F 1 "2.7K" H 8150 4850 50  0000 C CNN
-F 2 "" V 7930 4850 50  0001 C CNN
+F 1 "2.7K 1%" H 8200 4850 50  0000 C CNN
+F 2 "azonenberg_pcb:EIA_0402_RES_NOSILK" V 7930 4850 50  0001 C CNN
 F 3 "" H 8000 4850 50  0001 C CNN
 	1    8000 4850
@@
 P 8600 3900
 F 0 "R52" H 8450 3900 50  0000 C CNN
-F 1 "470" H 8750 3900 50  0000 C CNN
-F 2 "" V 8530 3900 50  0001 C CNN
+F 1 "470 1%" H 8800 3900 50  0000 C CNN
+F 2 "azonenberg_pcb:EIA_0402_RES_NOSILK" V 8530 3900 50  0001 C CNN
 F 3 "" H 8600 3900 50  0001 C CNN
 	1    8600 3900
@@
 F 0 "Q2" H 9450 4050 50  0000 L CNN
 F 1 "2SA2039-TL-E" H 9450 4150 50  0000 L CNN
-F 2 "" H 9450 4200 50  0001 C CNN
+F 2 "azonenberg_pcb:TO_253" H 9450 4200 50  0001 C CNN
 F 3 "" H 9250 4100 50  0001 C CNN
 	1    9250 4100
@@
 F 0 "R58" H 3000 5050 50  0000 C CNN
 F 1 "49.9K 1%" H 3100 5250 50  0000 C CNN
-F 2 "" V 3030 5050 50  0001 C CNN
+F 2 "azonenberg_pcb:EIA_0402_RES_NOSILK" V 3030 5050 50  0001 C CNN
 F 3 "" H 3100 5050 50  0001 C CNN
 	1    3100 5050
@@
 Wire Wire Line
 	2400 1100 2500 1100
+$Comp
+L device:R R57
+U 1 1 5E8EA1D4
+P 6600 5300
+F 0 "R57" H 6500 5300 50  0000 C CNN
+F 1 "49.9K 1%" H 6600 5100 50  0000 C CNN
+F 2 "azonenberg_pcb:EIA_0402_RES_NOSILK" V 6530 5300 50  0001 C CNN
+F 3 "" H 6600 5300 50  0001 C CNN
+	1    6600 5300
+	1    0    0    -1
+$EndComp
 $EndSCHEMATC
