File: boards/MAXWELL/maxwell-main/rightpods.sch (KiCad schematic (older format))
At the start: 14 parts

Commit message: Left pods
Parts:
- gave numbers to parts that had none: 7
Connections:
- net K7_CLK_N: now also U2.D10 (IO_L12N_T1_MRCC_16); no longer U2.C12 (IO_L13P_T2_MRCC_16)
- net K7_CLK_P: now also U2.E10 (IO_L12P_T1_MRCC_16); no longer U2.D10 (IO_L12N_T1_MRCC_16)
- net POD10_D0_N: now also U2.C11 (IO_L13N_T2_MRCC_16); no longer U2.A8 (IO_L9N_T1_DQS_16)
- net POD10_D0_P: now also U2.C12 (IO_L13P_T2_MRCC_16); no longer U2.A9 (IO_L9P_T1_DQS_16)
- net POD10_D1_N: now also U2.D8 (IO_L8N_T1_16); no longer U2.B9 (IO_L10N_T1_16)
- net POD10_D1_P: now also U2.D9 (IO_L8P_T1_16); no longer U2.C9 (IO_L10P_T1_16)
- net POD10_D2_N: now also U2.A8 (IO_L9N_T1_DQS_16); no longer U2.F10 (IO_L11N_T1_SRCC_16)
- net POD10_D2_P: now also U2.A9 (IO_L9P_T1_DQS_16); no longer U2.G11 (IO_L11P_T1_SRCC_16)
- net POD10_D3_N: now also U2.B9 (IO_L10N_T1_16); no longer U2.C11 (IO_L13N_T2_MRCC_16)
- net POD10_D3_P: now also U2.C9 (IO_L10P_T1_16); no longer U2.E10 (IO_L12P_T1_MRCC_16)
- net POD10_D4_N: now also U2.F13 (IO_L15N_T2_DQS_16); no longer U2.D11 (IO_L14N_T2_SRCC_16)
- net POD10_D4_P: now also U2.F14 (IO_L15P_T2_DQS_16); no longer U2.E11 (IO_L14P_T2_SRCC_16)
- net POD10_D5_N: now also U2.F12 (IO_L16N_T2_16); no longer U2.F13 (IO_L15N_T2_DQS_16)
- net POD10_D5_P: now also U2.G12 (IO_L16P_T2_16); no longer U2.F14 (IO_L15P_T2_DQS_16)
- net POD10_D6_N: now also U2.D13 (IO_L17N_T2_16); no longer U2.F12 (IO_L16N_T2_16)
- net POD10_D6_P: now also U2.D14 (IO_L17P_T2_16); no longer U2.G12 (IO_L16P_T2_16)
- net POD10_D7_N: now also U2.E12 (IO_L18N_T2_16); no longer U2.D13 (IO_L17N_T2_16)
- net POD10_D7_P: now also U2.E13 (IO_L18P_T2_16); no longer U2.D14 (IO_L17P_T2_16)
- net POD11_D0_N: now also U2.D11 (IO_L14N_T2_SRCC_16); no longer U2.E12 (IO_L18N_T2_16)
- net POD11_D0_P: now also U2.E11 (IO_L14P_T2_SRCC_16); no longer U2.E13 (IO_L18P_T2_16)
- net POD6_D0_N: now also U2.F18 (IO_L11N_T1_SRCC_AD12N_15); no longer U2.B16 (IO_L1N_T0_AD0N_15)
- net POD6_D0_P: now also U2.G17 (IO_L11P_T1_SRCC_AD12P_15); no longer U2.C16 (IO_L1P_T0_AD0P_15)
- net POD6_D1_N: now also U2.B16 (IO_L1N_T0_AD0N_15); no longer U2.A19 (IO_L2N_T0_AD8N_15)
- net POD6_D1_P: now also U2.C16 (IO_L1P_T0_AD0P_15); no longer U2.A18 (IO_L2P_T0_AD8P_15)
- net POD6_D2_N: now also U2.A19 (IO_L2N_T0_AD8N_15); no longer U2.A17 (IO_L3N_T0_DQS_AD1N_15)
- net POD6_D2_P: now also U2.A18 (IO_L2P_T0_AD8P_15); no longer U2.B17 (IO_L3P_T0_DQS_AD1P_15)
- net POD6_D3_N: now also U2.A17 (IO_L3N_T0_DQS_AD1N_15); no longer U2.B19 (IO_L4N_T0_AD9N_15)
- net POD6_D3_P: now also U2.B17 (IO_L3P_T0_DQS_AD1P_15); no longer U2.C19 (IO_L4P_T0_AD9P_15)
- net POD6_D4_N: now also U2.B19 (IO_L4N_T0_AD9N_15); no longer U2.C18 (IO_L5N_T0_AD2N_15)
- net POD6_D4_P: now also U2.C19 (IO_L4P_T0_AD9P_15); no longer U2.C17 (IO_L5P_T0_AD2P_15)
- net POD6_D5_N: now also U2.C18 (IO_L5N_T0_AD2N_15); no longer U2.D16 (IO_L6N_T0_VREF_15)
- net POD6_D5_P: now also U2.C17 (IO_L5P_T0_AD2P_15); no longer U2.D15 (IO_L6P_T0_15)
- net POD6_D6_N: now also U2.D16 (IO_L6N_T0_VREF_15); no longer U2.G16 (IO_L7N_T1_AD10N_15)
- net POD6_D6_P: now also U2.D15 (IO_L6P_T0_15); no longer U2.H16 (IO_L7P_T1_AD10P_15)
- net POD6_D7_N: now also U2.G16 (IO_L7N_T1_AD10N_15); no longer U2.F15 (IO_L8N_T1_AD3N_15)
- net POD6_D7_P: now also U2.H16 (IO_L7P_T1_AD10P_15); no longer U2.G15 (IO_L8P_T1_AD3P_15)
- net POD7_D0_N: now also U2.E17 (IO_L12N_T1_MRCC_AD5N_15); no longer U2.J16 (IO_L9N_T1_DQS_AD11N_15)
- net POD7_D0_P: now also U2.F17 (IO_L12P_T1_MRCC_AD5P_15); no longer U2.J15 (IO_L9P_T1_DQS_AD11P_15)
- net POD7_D1_N: now also U2.F15 (IO_L8N_T1_AD3N_15); no longer U2.E16 (IO_L10N_T1_AD4N_15)
- net POD7_D1_P: now also U2.G15 (IO_L8P_T1_AD3P_15); no longer U2.E15 (IO_L10P_T1_AD4P_15)
- net POD7_D2_N: now also U2.J16 (IO_L9N_T1_DQS_AD11N_15); no longer U2.F18 (IO_L11N_T1_SRCC_AD12N_15)
- net POD7_D2_P: now also U2.J15 (IO_L9P_T1_DQS_AD11P_15); no longer U2.G17 (IO_L11P_T1_SRCC_AD12P_15)
- net POD7_D3_N: now also U2.E16 (IO_L10N_T1_AD4N_15); no longer U2.E17 (IO_L12N_T1_MRCC_AD5N_15)
- net POD7_D3_P: now also U2.E15 (IO_L10P_T1_AD4P_15); no longer U2.F17 (IO_L12P_T1_MRCC_AD5P_15)
- net POD7_D4_N: now also U2.H18 (IO_L14N_T2_SRCC_15); no longer U2.D18 (IO_L13N_T2_MRCC_15)
- net POD7_D4_P: now also U2.H17 (IO_L14P_T2_SRCC_15); no longer U2.E18 (IO_L13P_T2_MRCC_15)
- net POD7_D5_N: now also U2.D20 (IO_L15N_T2_DQS_ADV_B_15); no longer U2.H18 (IO_L14N_T2_SRCC_15)
- net POD7_D5_P: now also U2.D19 (IO_L15P_T2_DQS_15); no longer U2.H17 (IO_L14P_T2_SRCC_15)
- net POD7_D6_N: now also U2.F20 (IO_L16N_T2_A27_15); no longer U2.D20 (IO_L15N_T2_DQS_ADV_B_15)
- net POD7_D6_P: now also U2.G19 (IO_L16P_T2_A28_15); no longer U2.D19 (IO_L15P_T2_DQS_15)
- net POD7_D7_N: now also U2.E20 (IO_L17N_T2_A25_15); no longer U2.F20 (IO_L16N_T2_A27_15)
- net POD7_D7_P: now also U2.F19 (IO_L17P_T2_A26_15); no longer U2.G19 (IO_L16P_T2_A28_15)
- net POD8_D0_N: now also U2.D18 (IO_L13N_T2_MRCC_15); no longer U2.E20 (IO_L17N_T2_A25_15)
- net POD8_D0_P: now also U2.E18 (IO_L13P_T2_MRCC_15); no longer U2.F19 (IO_L17P_T2_A26_15)
- net POD9_D0_N: now also U2.F10 (IO_L11N_T1_SRCC_16); no longer U2.H8 (IO_L1N_T0_16)
- net POD9_D0_P: now also U2.G11 (IO_L11P_T1_SRCC_16); no longer U2.H9 (IO_L1P_T0_16)
- net POD9_D1_N: now also U2.H8 (IO_L1N_T0_16); no longer U2.G9 (IO_L2N_T0_16)
- net POD9_D1_P: now also U2.H9 (IO_L1P_T0_16); no longer U2.G10 (IO_L2P_T0_16)
- net POD9_D2_N: now also U2.G9 (IO_L2N_T0_16); no longer U2.H13 (IO_L3N_T0_DQS_16)
- net POD9_D2_P: now also U2.G10 (IO_L2P_T0_16); no longer U2.J13 (IO_L3P_T0_DQS_16)
- net POD9_D3_N: now also U2.H13 (IO_L3N_T0_DQS_16); no longer U2.J10 (IO_L4N_T0_16)
- net POD9_D3_P: now also U2.J13 (IO_L3P_T0_DQS_16); no longer U2.J11 (IO_L4P_T0_16)
- net POD9_D4_N: now also U2.J10 (IO_L4N_T0_16); no longer U2.G14 (IO_L5N_T0_16)
- net POD9_D4_P: now also U2.J11 (IO_L4P_T0_16); no longer U2.H14 (IO_L5P_T0_16)
- net POD9_D5_N: now also U2.G14 (IO_L5N_T0_16); no longer U2.H11 (IO_L6N_T0_VREF_16)
- net POD9_D5_P: now also U2.H14 (IO_L5P_T0_16); no longer U2.H12 (IO_L6P_T0_16)
- net POD9_D6_N: now also U2.H11 (IO_L6N_T0_VREF_16); no longer U2.F8 (IO_L7N_T1_16)
- net POD9_D6_P: now also U2.H12 (IO_L6P_T0_16); no longer U2.F9 (IO_L7P_T1_16)
- net POD9_D7_N: now also U2.F8 (IO_L7N_T1_16); no longer U2.D8 (IO_L8N_T1_16)
- net POD9_D7_P: now also U2.F9 (IO_L7P_T1_16); no longer U2.D9 (IO_L8P_T1_16)
Changed lines of the file:
@@
 AR Path="/5EDD71F2/5F2ECCDE" Ref="U?"  Part="9"
 AR Path="/5EDD723A/5F2ECCDE" Ref="U?"  Part="6"
-AR Path="/5EDD723A/5F2BB4CD/5F2ECCDE" Ref="U?"  Part="7"
-F 0 "U?" H 10800 9200 50  0000 L CNN
+AR Path="/5EDD723A/5F2BB4CD/5F2ECCDE" Ref="U2"  Part="7"
+F 0 "U2" H 10800 9200 50  0000 L CNN
 F 1 "XC7K160T-2FFG676C" H 10800 9100 50  0000 L CNN
 F 2 "" H 10800 9250 50  0001 C CNN
@@
 AR Path="/5EDD71F2/5F2ECCE4" Ref="U?"  Part="9"
 AR Path="/5EDD723A/5F2ECCE4" Ref="U?"  Part="8"
-AR Path="/5EDD723A/5F2BB4CD/5F2ECCE4" Ref="U?"  Part="8"
-F 0 "U?" H 13600 9200 50  0000 L CNN
+AR Path="/5EDD723A/5F2BB4CD/5F2ECCE4" Ref="U2"  Part="8"
+F 0 "U2" H 13600 9200 50  0000 L CNN
 F 1 "XC7K160T-2FFG676C" H 13600 9100 50  0000 L CNN
 F 2 "" H 13600 9250 50  0001 C CNN
@@
 $EndSheet
 $Comp
-L special-azonenberg:CONN_SFF8087 J?
+L special-azonenberg:CONN_SFF8087 J3
 U 1 1 5F3DFECC
 P 1550 5650
-F 0 "J?" H 1550 5600 50  0000 L CNN
+F 0 "J3" H 1550 5600 50  0000 L CNN
 F 1 "CONN_SFF8087" H 1550 5500 50  0000 L CNN
 F 2 "" H 1550 5650 50  0001 C CNN
@@
 $EndComp
 $Comp
-L special-azonenberg:CONN_SFF8087 J?
+L special-azonenberg:CONN_SFF8087 J3
 U 2 1 5F3E0DC5
 P 1550 3200
-F 0 "J?" H 1550 3150 50  0000 L CNN
+F 0 "J3" H 1550 3150 50  0000 L CNN
 F 1 "CONN_SFF8087" H 1550 3050 50  0000 L CNN
 F 2 "" H 1550 3200 50  0001 C CNN
@@
 POD6_D7_N
 $Comp
-L special-azonenberg:CONN_SFF8087 J?
+L special-azonenberg:CONN_SFF8087 J4
 U 2 1 5F3EE49C
 P 2950 3200
-F 0 "J?" H 2950 3150 50  0000 L CNN
+F 0 "J4" H 2950 3150 50  0000 L CNN
 F 1 "CONN_SFF8087" H 2950 3050 50  0000 L CNN
 F 2 "" H 2950 3200 50  0001 C CNN
@@
 POD7_D7_N
 $Comp
-L special-azonenberg:CONN_SFF8087 J?
+L special-azonenberg:CONN_SFF8087 J5
 U 2 1 5F3F3B95
 P 4350 3200
-F 0 "J?" H 4350 3150 50  0000 L CNN
+F 0 "J5" H 4350 3150 50  0000 L CNN
 F 1 "CONN_SFF8087" H 4350 3050 50  0000 L CNN
 F 2 "" H 4350 3200 50  0001 C CNN
@@
 POD8_D7_N
 $Comp
-L special-azonenberg:CONN_SFF8087 J?
+L special-azonenberg:CONN_SFF8087 J6
 U 2 1 5F3F3BAF
 P 5750 3200
-F 0 "J?" H 5750 3150 50  0000 L CNN
+F 0 "J6" H 5750 3150 50  0000 L CNN
 F 1 "CONN_SFF8087" H 5750 3050 50  0000 L CNN
 F 2 "" H 5750 3200 50  0001 C CNN
@@
 Text Label 5650 3150 2    50   ~ 0
 POD9_D7_N
+Text Label 10600 4800 2    50   ~ 0
+POD6_D3_P
+Text Label 10600 4900 2    50   ~ 0
+POD6_D3_N
 Text Label 10600 5000 2    50   ~ 0
-POD6_D3_P
+POD6_D4_P
 Text Label 10600 5100 2    50   ~ 0
-POD6_D3_N
+POD6_D4_N
 Text Label 10600 5200 2    50   ~ 0
-POD6_D4_P
+POD6_D5_P
 Text Label 10600 5300 2    50   ~ 0
-POD6_D4_N
+POD6_D5_N
 Text Label 10600 5400 2    50   ~ 0
-POD6_D5_P
+POD6_D6_P
 Text Label 10600 5500 2    50   ~ 0
-POD6_D5_N
+POD6_D6_N
 Text Label 10600 5600 2    50   ~ 0
-POD6_D6_P
+POD6_D7_P
 Text Label 10600 5700 2    50   ~ 0
-POD6_D6_N
+POD6_D7_N
+Text Label 10600 6600 2    50   ~ 0
+POD7_D0_P
+Text Label 10600 6700 2    50   ~ 0
+POD7_D0_N
 Text Label 10600 5800 2    50   ~ 0
-POD6_D7_P
+POD7_D1_P
 Text Label 10600 5900 2    50   ~ 0
-POD6_D7_N
+POD7_D1_N
+Text Label 10600 6200 2    50   ~ 0
+POD7_D3_P
+Text Label 10600 6300 2    50   ~ 0
+POD7_D3_N
 Text Label 10600 6000 2    50   ~ 0
-POD7_D0_P
+POD7_D2_P
 Text Label 10600 6100 2    50   ~ 0
-POD7_D0_N
-Text Label 10600 6200 2    50   ~ 0
-POD7_D1_P
-Text Label 10600 6300 2    50   ~ 0
-POD7_D1_N
-Text Label 10600 6600 2    50   ~ 0
-POD7_D3_P
-Text Label 10600 6700 2    50   ~ 0
-POD7_D3_N
-Text Label 10600 6400 2    50   ~ 0
-POD7_D2_P
-Text Label 10600 6500 2    50   ~ 0
 POD7_D2_N
+Text Label 10600 7000 2    50   ~ 0
+POD7_D4_P
+Text Label 10600 7100 2    50   ~ 0
+POD7_D4_N
+Text Label 10600 7200 2    50   ~ 0
+POD7_D5_P
+Text Label 10600 7300 2    50   ~ 0
+POD7_D5_N
+Text Label 10600 7400 2    50   ~ 0
+POD7_D6_P
+Text Label 10600 7500 2    50   ~ 0
+POD7_D6_N
+Text Label 10600 7600 2    50   ~ 0
+POD7_D7_P
+Text Label 10600 7700 2    50   ~ 0
+POD7_D7_N
 Text Label 10600 6800 2    50   ~ 0
-POD7_D4_P
+POD8_D0_P
 Text Label 10600 6900 2    50   ~ 0
-POD7_D4_N
-Text Label 10600 7000 2    50   ~ 0
-POD7_D5_P
-Text Label 10600 7100 2    50   ~ 0
-POD7_D5_N
-Text Label 10600 7200 2    50   ~ 0
-POD7_D6_P
-Text Label 10600 7300 2    50   ~ 0
-POD7_D6_N
-Text Label 10600 7400 2    50   ~ 0
-POD7_D7_P
-Text Label 10600 7500 2    50   ~ 0
-POD7_D7_N
-Text Label 10600 7600 2    50   ~ 0
-POD8_D0_P
-Text Label 10600 7700 2    50   ~ 0
 POD8_D0_N
 Text Label 10600 7800 2    50   ~ 0
@@
 Text Label 10600 9100 2    50   ~ 0
 POD8_D7_N
+Text Label 13400 6400 2    50   ~ 0
+POD9_D0_P
+Text Label 13400 6500 2    50   ~ 0
+POD9_D0_N
 Text Label 13400 4400 2    50   ~ 0
-POD9_D0_P
+POD9_D1_P
 Text Label 13400 4500 2    50   ~ 0
-POD9_D0_N
+POD9_D1_N
+Text Label 13400 4800 2    50   ~ 0
+POD9_D3_P
+Text Label 13400 4900 2    50   ~ 0
+POD9_D3_N
 Text Label 13400 4600 2    50   ~ 0
-POD9_D1_P
+POD9_D2_P
 Text Label 13400 4700 2    50   ~ 0
-POD9_D1_N
+POD9_D2_N
 Text Label 13400 5000 2    50   ~ 0
-POD9_D3_P
+POD9_D4_P
 Text Label 13400 5100 2    50   ~ 0
-POD9_D3_N
-Text Label 13400 4800 2    50   ~ 0
-POD9_D2_P
-Text Label 13400 4900 2    50   ~ 0
-POD9_D2_N
+POD9_D4_N
 Text Label 13400 5200 2    50   ~ 0
-POD9_D4_P
+POD9_D5_P
 Text Label 13400 5300 2    50   ~ 0
-POD9_D4_N
+POD9_D5_N
 Text Label 13400 5400 2    50   ~ 0
-POD9_D5_P
+POD9_D6_P
 Text Label 13400 5500 2    50   ~ 0
-POD9_D5_N
+POD9_D6_N
 Text Label 13400 5600 2    50   ~ 0
-POD9_D6_P
+POD9_D7_P
 Text Label 13400 5700 2    50   ~ 0
-POD9_D6_N
-Text Label 13400 5800 2    50   ~ 0
-POD9_D7_P
-Text Label 13400 5900 2    50   ~ 0
 POD9_D7_N
 $Comp
-L special-azonenberg:CONN_SFF8087 J?
+L special-azonenberg:CONN_SFF8087 J7
 U 2 1 5F405F23
 P 7150 3200
-F 0 "J?" H 7150 3150 50  0000 L CNN
+F 0 "J7" H 7150 3150 50  0000 L CNN
 F 1 "CONN_SFF8087" H 7150 3050 50  0000 L CNN
 F 2 "" H 7150 3200 50  0001 C CNN
@@
 POD10_D7_N
 $Comp
-L special-azonenberg:CONN_SFF8087 J?
+L special-azonenberg:CONN_SFF8087 J8
 U 2 1 5F405F3D
 P 8550 3200
-F 0 "J?" H 8550 3150 50  0000 L CNN
+F 0 "J8" H 8550 3150 50  0000 L CNN
 F 1 "CONN_SFF8087" H 8550 3050 50  0000 L CNN
 F 2 "" H 8550 3200 50  0001 C CNN
@@
 Text Label 8450 3150 2    50   ~ 0
 POD11_D7_N
-Text Label 13400 7200 2    50   ~ 0
+Text Label 13400 7400 2    50   ~ 0
 POD10_D5_P
-Text Label 13400 7300 2    50   ~ 0
+Text Label 13400 7500 2    50   ~ 0
 POD10_D5_N
-Text Label 13400 7400 2    50   ~ 0
+Text Label 13400 7600 2    50   ~ 0
 POD10_D6_P
-Text Label 13400 7500 2    50   ~ 0
+Text Label 13400 7700 2    50   ~ 0
 POD10_D6_N
-Text Label 13400 7600 2    50   ~ 0
+Text Label 13400 7800 2    50   ~ 0
 POD10_D7_P
-Text Label 13400 7700 2    50   ~ 0
+Text Label 13400 7900 2    50   ~ 0
 POD10_D7_N
-Text Label 13400 7800 2    50   ~ 0
+Text Label 13400 7000 2    50   ~ 0
 POD11_D0_P
-Text Label 13400 7900 2    50   ~ 0
+Text Label 13400 7100 2    50   ~ 0
 POD11_D0_N
 Text Label 13400 8000 2    50   ~ 0
@@
 Text Label 13500 2000 2    50   ~ 0
 POD11_D7_N
-Text Label 10600 4900 2    50   ~ 0
+Text Label 10600 4700 2    50   ~ 0
 POD6_D2_N
-Text Label 10600 4800 2    50   ~ 0
+Text Label 10600 4600 2    50   ~ 0
 POD6_D2_P
-Text Label 10600 4700 2    50   ~ 0
+Text Label 10600 4500 2    50   ~ 0
 POD6_D1_N
-Text Label 10600 4600 2    50   ~ 0
+Text Label 10600 4400 2    50   ~ 0
 POD6_D1_P
-Text Label 10600 4500 2    50   ~ 0
+Text Label 10600 6500 2    50   ~ 0
 POD6_D0_N
-Text Label 10600 4400 2    50   ~ 0
+Text Label 10600 6400 2    50   ~ 0
 POD6_D0_P
-Text Label 13400 7100 2    50   ~ 0
+Text Label 13400 7300 2    50   ~ 0
 POD10_D4_N
-Text Label 13400 7000 2    50   ~ 0
+Text Label 13400 7200 2    50   ~ 0
 POD10_D4_P
-Text Label 13400 6500 2    50   ~ 0
+Text Label 13400 6100 2    50   ~ 0
 POD10_D2_N
-Text Label 13400 6400 2    50   ~ 0
+Text Label 13400 6000 2    50   ~ 0
 POD10_D2_P
+Text Label 13400 6300 2    50   ~ 0
+POD10_D3_N
+Text Label 13400 6200 2    50   ~ 0
+POD10_D3_P
+Text Label 13400 5900 2    50   ~ 0
+POD10_D1_N
+Text Label 13400 5800 2    50   ~ 0
+POD10_D1_P
 Text Label 13400 6900 2    50   ~ 0
-POD10_D3_N
-Text Label 13400 6600 2    50   ~ 0
-POD10_D3_P
-Text Label 13400 6300 2    50   ~ 0
-POD10_D1_N
-Text Label 13400 6200 2    50   ~ 0
-POD10_D1_P
-Text Label 13400 6100 2    50   ~ 0
 POD10_D0_N
-Text Label 13400 6000 2    50   ~ 0
+Text Label 13400 6800 2    50   ~ 0
 POD10_D0_P
+Text HLabel 13400 6600 0    50   Input ~ 0
+K7_CLK_P
 Text HLabel 13400 6700 0    50   Input ~ 0
-K7_CLK_P
-Text HLabel 13400 6800 0    50   Input ~ 0
 K7_CLK_N
 $Comp
-L special-azonenberg:CONN_SFF8087 J?
+L special-azonenberg:CONN_SFF8087 J4
 U 1 1 5F4F0590
 P 2950 5650
-F 0 "J?" H 2950 5600 50  0000 L CNN
+F 0 "J4" H 2950 5600 50  0000 L CNN
 F 1 "CONN_SFF8087" H 2950 5500 50  0000 L CNN
 F 2 "" H 2950 5650 50  0001 C CNN
@@
 $EndComp
 $Comp
-L special-azonenberg:CONN_SFF8087 J?
+L special-azonenberg:CONN_SFF8087 J5
 U 1 1 5F4F181F
 P 4350 5650
-F 0 "J?" H 4350 5600 50  0000 L CNN
+F 0 "J5" H 4350 5600 50  0000 L CNN
 F 1 "CONN_SFF8087" H 4350 5500 50  0000 L CNN
 F 2 "" H 4350 5650 50  0001 C CNN
@@
 $EndComp
 $Comp
-L special-azonenberg:CONN_SFF8087 J?
+L special-azonenberg:CONN_SFF8087 J6
 U 1 1 5F4F28DA
 P 5750 5650
-F 0 "J?" H 5750 5600 50  0000 L CNN
+F 0 "J6" H 5750 5600 50  0000 L CNN
 F 1 "CONN_SFF8087" H 5750 5500 50  0000 L CNN
 F 2 "" H 5750 5650 50  0001 C CNN
@@
 $EndComp
 $Comp
-L special-azonenberg:CONN_SFF8087 J?
+L special-azonenberg:CONN_SFF8087 J7
 U 1 1 5F4F3578
 P 7150 5650
-F 0 "J?" H 7150 5600 50  0000 L CNN
+F 0 "J7" H 7150 5600 50  0000 L CNN
 F 1 "CONN_SFF8087" H 7150 5500 50  0000 L CNN
 F 2 "" H 7150 5650 50  0001 C CNN
@@
 $EndComp
 $Comp
-L special-azonenberg:CONN_SFF8087 J?
+L special-azonenberg:CONN_SFF8087 J8
 U 1 1 5F4F4453
 P 8550 5650
-F 0 "J?" H 8550 5600 50  0000 L CNN
+F 0 "J8" H 8550 5600 50  0000 L CNN
 F 1 "CONN_SFF8087" H 8550 5500 50  0000 L CNN
 F 2 "" H 8550 5650 50  0001 C CNN
