File: boards/MAXWELL/maxwell-main/inputs.sch (KiCad schematic (older format))
At the start: 1 part, among them U4 XC7S6-1FTGB196C

Commit message: Changed comparators on GTX inputs to ADCMP582s, added pins for 0V5 supply
Changed lines of the file:
@@
 $Descr A4 11693 8268
 encoding utf-8
-Sheet 6 18
+Sheet 7 18
 Title "MAXWELL Main Board"
 Date "2020-06-20"
@@
 F39 "GTX_TRIG_OUT_N" O L 5000 4350 50
 F40 "1V2" I R 6350 1450 50
+F41 "0V5" I L 5000 1450 50
+F42 "5V0" I L 5000 1350 50
+F43 "5V0_N" I L 5000 1550 50
 $EndSheet
 Text Label 9100 1350 2    50   ~ 0
@@
 Text Label 1400 1350 2    50   ~ 0
 GND
+Text HLabel 5000 1350 0    50   Input ~ 0
+5V0
+Text HLabel 5000 1450 0    50   Input ~ 0
+0V5
+Text HLabel 5000 1550 0    50   Input ~ 0
+5V0_N
 $EndSCHEMATC
