File: boards/MAXWELL/maxwell-main/rgmii.sch (KiCad schematic (older format))
At the start: 54 parts, among them J11 BEL_FUSE_0826-1G1T-23-F, U2 XC7K160T-2FFG676C, U35 KSZ9031RN, U39 AT24MAC402-UDFN

Commit message: Began assigning IC footprints
Parts:
- U2: footprint (none) -> azonenberg_pcb:BGA_676_27x27_FULLARRAY_1MM_FFG676
Changed lines of the file:
@@
 F 0 "U2" H 2250 5900 50  0000 L CNN
 F 1 "XC7K160T-2FFG676C" H 2250 5800 50  0000 L CNN
-F 2 "" H 2250 5950 50  0001 C CNN
+F 2 "azonenberg_pcb:BGA_676_27x27_FULLARRAY_1MM_FFG676" H 2250 5950 50  0001 C CNN
 F 3 "" H 2250 5950 50  0001 C CNN
 	6    2250 5950
