File: boards/MAXWELL/maxwell-main/iofpga.sch (KiCad schematic (older format))
At the start: 39 parts, among them J2 XILINX_JTAG, U29 S25FL128LAGNFV010, U4 XC7S6-1FTGB196C

Commit message: Continued schematic review. Added footprints for C1-C282.
Parts:
- C37, C40: footprint (none) -> azonenberg_pcb:EIA_1210_CAP_NOSILK
- C38, C44, C46, C47, C53, C58, C62, C63: footprint (none) -> azonenberg_pcb:EIA_0603_CAP_NOSILK
- C39: footprint (none) -> azonenberg_pcb:EIA_0805_CAP_NOSILK
- C41, C42, C43, C45, C48, C49, C50, C51, C52, C54, C55, C56, C57, C59, C60, C61, C64: footprint (none) -> azonenberg_pcb:EIA_0402_CAP_NOSILK
Changed lines of the file:
@@
 F 0 "U29" H 8950 5137 60  0000 C CNN
 F 1 "S25FL128LAGNFV010" H 8950 5031 60  0000 C CNN
-F 2 "" H 8950 4450 60  0000 C CNN
+F 2 "" H 8950 4450 60  0001 C CNN
 F 3 "" H 8950 4450 60  0000 C CNN
 	1    8950 4450
@@
 F 0 "J2" H 3169 8258 60  0000 L CNN
 F 1 "XILINX_JTAG" H 3169 8152 60  0000 L CNN
-F 2 "" H 2450 7550 60  0000 C CNN
+F 2 "" H 2450 7550 60  0001 C CNN
 F 3 "" H 2450 7550 60  0000 C CNN
 	1    2450 7550
@@
 F 0 "C37" H 4865 3596 50  0000 L CNN
 F 1 "100 uF" H 4865 3505 50  0000 L CNN
-F 2 "" H 4788 3400 50  0001 C CNN
+F 2 "azonenberg_pcb:EIA_1210_CAP_NOSILK" H 4788 3400 50  0001 C CNN
 F 3 "" H 4750 3550 50  0001 C CNN
 	1    4750 3550
@@
 F 0 "C44" H 5415 3596 50  0000 L CNN
 F 1 "4.7 uF" H 5415 3505 50  0000 L CNN
-F 2 "" H 5338 3400 50  0001 C CNN
+F 2 "azonenberg_pcb:EIA_0603_CAP_NOSILK" H 5338 3400 50  0001 C CNN
 F 3 "" H 5300 3550 50  0001 C CNN
 	1    5300 3550
@@
 F 0 "C51" H 5915 3596 50  0000 L CNN
 F 1 "0.47 uF" H 5915 3505 50  0000 L CNN
-F 2 "" H 5838 3400 50  0001 C CNN
+F 2 "azonenberg_pcb:EIA_0402_CAP_NOSILK" H 5838 3400 50  0001 C CNN
 F 3 "" H 5800 3550 50  0001 C CNN
 	1    5800 3550
@@
 F 0 "C63" H 8615 4946 50  0000 L CNN
 F 1 "4.7 uF" H 8615 4855 50  0000 L CNN
-F 2 "" H 8538 4750 50  0001 C CNN
+F 2 "azonenberg_pcb:EIA_0603_CAP_NOSILK" H 8538 4750 50  0001 C CNN
 F 3 "" H 8500 4900 50  0001 C CNN
 	1    8500 4900
@@
 F 0 "C64" H 9115 4946 50  0000 L CNN
 F 1 "0.47 uF" H 9115 4855 50  0000 L CNN
-F 2 "" H 9038 4750 50  0001 C CNN
+F 2 "azonenberg_pcb:EIA_0402_CAP_NOSILK" H 9038 4750 50  0001 C CNN
 F 3 "" H 9000 4900 50  0001 C CNN
 	1    9000 4900
@@
 F 0 "C38" H 4865 4096 50  0000 L CNN
 F 1 "4.7 uF" H 4865 4005 50  0000 L CNN
-F 2 "" H 4788 3900 50  0001 C CNN
+F 2 "azonenberg_pcb:EIA_0603_CAP_NOSILK" H 4788 3900 50  0001 C CNN
 F 3 "" H 4750 4050 50  0001 C CNN
 	1    4750 4050
@@
 F 0 "C45" H 5415 4096 50  0000 L CNN
 F 1 "0.47 uF" H 5415 4005 50  0000 L CNN
-F 2 "" H 5338 3900 50  0001 C CNN
+F 2 "azonenberg_pcb:EIA_0402_CAP_NOSILK" H 5338 3900 50  0001 C CNN
 F 3 "" H 5300 4050 50  0001 C CNN
 	1    5300 4050
@@
 F 0 "C39" H 4865 4696 50  0000 L CNN
 F 1 "47 uF" H 4865 4605 50  0000 L CNN
-F 2 "" H 4788 4500 50  0001 C CNN
+F 2 "azonenberg_pcb:EIA_0805_CAP_NOSILK" H 4788 4500 50  0001 C CNN
 F 3 "" H 4750 4650 50  0001 C CNN
 	1    4750 4650
@@
 F 0 "C46" H 5415 4696 50  0000 L CNN
 F 1 "4.7 uF" H 5415 4605 50  0000 L CNN
-F 2 "" H 5338 4500 50  0001 C CNN
+F 2 "azonenberg_pcb:EIA_0603_CAP_NOSILK" H 5338 4500 50  0001 C CNN
 F 3 "" H 5300 4650 50  0001 C CNN
 	1    5300 4650
@@
 F 0 "C52" H 5915 4696 50  0000 L CNN
 F 1 "0.47 uF" H 5915 4605 50  0000 L CNN
-F 2 "" H 5838 4500 50  0001 C CNN
+F 2 "azonenberg_pcb:EIA_0402_CAP_NOSILK" H 5838 4500 50  0001 C CNN
 F 3 "" H 5800 4650 50  0001 C CNN
 	1    5800 4650
@@
 F 0 "C57" H 6465 4696 50  0000 L CNN
 F 1 "0.47 uF" H 6465 4605 50  0000 L CNN
-F 2 "" H 6388 4500 50  0001 C CNN
+F 2 "azonenberg_pcb:EIA_0402_CAP_NOSILK" H 6388 4500 50  0001 C CNN
 F 3 "" H 6350 4650 50  0001 C CNN
 	1    6350 4650
@@
 F 0 "C40" H 4865 5246 50  0000 L CNN
 F 1 "100 uF" H 4865 5155 50  0000 L CNN
-F 2 "" H 4788 5050 50  0001 C CNN
+F 2 "azonenberg_pcb:EIA_1210_CAP_NOSILK" H 4788 5050 50  0001 C CNN
 F 3 "" H 4750 5200 50  0001 C CNN
 	1    4750 5200
@@
 F 0 "C47" H 5415 5246 50  0000 L CNN
 F 1 "4.7 uF" H 5415 5155 50  0000 L CNN
-F 2 "" H 5338 5050 50  0001 C CNN
+F 2 "azonenberg_pcb:EIA_0603_CAP_NOSILK" H 5338 5050 50  0001 C CNN
 F 3 "" H 5300 5200 50  0001 C CNN
 	1    5300 5200
@@
 F 0 "C53" H 5915 5246 50  0000 L CNN
 F 1 "4.7 uF" H 5915 5155 50  0000 L CNN
-F 2 "" H 5838 5050 50  0001 C CNN
+F 2 "azonenberg_pcb:EIA_0603_CAP_NOSILK" H 5838 5050 50  0001 C CNN
 F 3 "" H 5800 5200 50  0001 C CNN
 	1    5800 5200
@@
 F 0 "C58" H 6465 5246 50  0000 L CNN
 F 1 "4.7 uF" H 6465 5155 50  0000 L CNN
-F 2 "" H 6388 5050 50  0001 C CNN
+F 2 "azonenberg_pcb:EIA_0603_CAP_NOSILK" H 6388 5050 50  0001 C CNN
 F 3 "" H 6350 5200 50  0001 C CNN
 	1    6350 5200
@@
 F 0 "C62" H 6965 5246 50  0000 L CNN
 F 1 "4.7 uF" H 6965 5155 50  0000 L CNN
-F 2 "" H 6888 5050 50  0001 C CNN
+F 2 "azonenberg_pcb:EIA_0603_CAP_NOSILK" H 6888 5050 50  0001 C CNN
 F 3 "" H 6850 5200 50  0001 C CNN
 	1    6850 5200
@@
 F 0 "C41" H 4865 5696 50  0000 L CNN
 F 1 "0.47 uF" H 4865 5605 50  0000 L CNN
-F 2 "" H 4788 5500 50  0001 C CNN
+F 2 "azonenberg_pcb:EIA_0402_CAP_NOSILK" H 4788 5500 50  0001 C CNN
 F 3 "" H 4750 5650 50  0001 C CNN
 	1    4750 5650
@@
 F 0 "C48" H 5415 5696 50  0000 L CNN
 F 1 "0.47 uF" H 5415 5605 50  0000 L CNN
-F 2 "" H 5338 5500 50  0001 C CNN
+F 2 "azonenberg_pcb:EIA_0402_CAP_NOSILK" H 5338 5500 50  0001 C CNN
 F 3 "" H 5300 5650 50  0001 C CNN
 	1    5300 5650
@@
 F 0 "C54" H 5915 5696 50  0000 L CNN
 F 1 "0.47 uF" H 5915 5605 50  0000 L CNN
-F 2 "" H 5838 5500 50  0001 C CNN
+F 2 "azonenberg_pcb:EIA_0402_CAP_NOSILK" H 5838 5500 50  0001 C CNN
 F 3 "" H 5800 5650 50  0001 C CNN
 	1    5800 5650
@@
 F 0 "C59" H 6465 5696 50  0000 L CNN
 F 1 "0.47 uF" H 6465 5605 50  0000 L CNN
-F 2 "" H 6388 5500 50  0001 C CNN
+F 2 "azonenberg_pcb:EIA_0402_CAP_NOSILK" H 6388 5500 50  0001 C CNN
 F 3 "" H 6350 5650 50  0001 C CNN
 	1    6350 5650
@@
 F 0 "C42" H 4865 6146 50  0000 L CNN
 F 1 "0.47 uF" H 4865 6055 50  0000 L CNN
-F 2 "" H 4788 5950 50  0001 C CNN
+F 2 "azonenberg_pcb:EIA_0402_CAP_NOSILK" H 4788 5950 50  0001 C CNN
 F 3 "" H 4750 6100 50  0001 C CNN
 	1    4750 6100
@@
 F 0 "C49" H 5415 6146 50  0000 L CNN
 F 1 "0.47 uF" H 5415 6055 50  0000 L CNN
-F 2 "" H 5338 5950 50  0001 C CNN
+F 2 "azonenberg_pcb:EIA_0402_CAP_NOSILK" H 5338 5950 50  0001 C CNN
 F 3 "" H 5300 6100 50  0001 C CNN
 	1    5300 6100
@@
 F 0 "C55" H 5915 6146 50  0000 L CNN
 F 1 "0.47 uF" H 5915 6055 50  0000 L CNN
-F 2 "" H 5838 5950 50  0001 C CNN
+F 2 "azonenberg_pcb:EIA_0402_CAP_NOSILK" H 5838 5950 50  0001 C CNN
 F 3 "" H 5800 6100 50  0001 C CNN
 	1    5800 6100
@@
 F 0 "C60" H 6465 6146 50  0000 L CNN
 F 1 "0.47 uF" H 6465 6055 50  0000 L CNN
-F 2 "" H 6388 5950 50  0001 C CNN
+F 2 "azonenberg_pcb:EIA_0402_CAP_NOSILK" H 6388 5950 50  0001 C CNN
 F 3 "" H 6350 6100 50  0001 C CNN
 	1    6350 6100
@@
 F 0 "C43" H 4865 6596 50  0000 L CNN
 F 1 "0.47 uF" H 4865 6505 50  0000 L CNN
-F 2 "" H 4788 6400 50  0001 C CNN
+F 2 "azonenberg_pcb:EIA_0402_CAP_NOSILK" H 4788 6400 50  0001 C CNN
 F 3 "" H 4750 6550 50  0001 C CNN
 	1    4750 6550
@@
 F 0 "C50" H 5415 6596 50  0000 L CNN
 F 1 "0.47 uF" H 5415 6505 50  0000 L CNN
-F 2 "" H 5338 6400 50  0001 C CNN
+F 2 "azonenberg_pcb:EIA_0402_CAP_NOSILK" H 5338 6400 50  0001 C CNN
 F 3 "" H 5300 6550 50  0001 C CNN
 	1    5300 6550
@@
 F 0 "C56" H 5915 6596 50  0000 L CNN
 F 1 "0.47 uF" H 5915 6505 50  0000 L CNN
-F 2 "" H 5838 6400 50  0001 C CNN
+F 2 "azonenberg_pcb:EIA_0402_CAP_NOSILK" H 5838 6400 50  0001 C CNN
 F 3 "" H 5800 6550 50  0001 C CNN
 	1    5800 6550
@@
 F 0 "C61" H 6465 6596 50  0000 L CNN
 F 1 "0.47 uF" H 6465 6505 50  0000 L CNN
-F 2 "" H 6388 6400 50  0001 C CNN
+F 2 "azonenberg_pcb:EIA_0402_CAP_NOSILK" H 6388 6400 50  0001 C CNN
 F 3 "" H 6350 6550 50  0001 C CNN
 	1    6350 6550

Commit message: Continued schematic review. Finished verifying pinouts. Assigned lots more footprints.
Parts:
- J2: footprint (none) -> azonenberg_pcb:XILINX_JTAG_PTH_MOLEX_0878311420
Changed lines of the file:
@@
 F 0 "J2" H 3169 8258 60  0000 L CNN
 F 1 "XILINX_JTAG" H 3169 8152 60  0000 L CNN
-F 2 "" H 2450 7550 60  0001 C CNN
+F 2 "azonenberg_pcb:XILINX_JTAG_PTH_MOLEX_0878311420" H 2450 7550 60  0001 C CNN
 F 3 "" H 2450 7550 60  0000 C CNN
 	1    2450 7550

Commit message: Assigned footprints for all resistors
Parts:
- R25, R26, R27, R28, R29, R30, R31, R32: footprint (none) -> azonenberg_pcb:EIA_0402_RES_NOSILK
Changed lines of the file:
@@
 Sheet 9 18
 Title "MAXWELL Main Board"
-Date "2020-06-22"
+Date "2020-06-23"
 Rev "0.1"
 Comp "Antikernel Labs"
@@
 F 0 "R29" V 8000 3900 50  0000 C CNN
 F 1 "33" V 8050 4150 50  0000 C CNN
-F 2 "" V 7980 4150 50  0001 C CNN
+F 2 "azonenberg_pcb:EIA_0402_RES_NOSILK" V 7980 4150 50  0001 C CNN
 F 3 "" H 8050 4150 50  0001 C CNN
 	1    8050 4150
@@
 F 0 "R30" V 8000 4000 50  0000 C CNN
 F 1 "33" V 8050 4250 50  0000 C CNN
-F 2 "" V 7980 4250 50  0001 C CNN
+F 2 "azonenberg_pcb:EIA_0402_RES_NOSILK" V 7980 4250 50  0001 C CNN
 F 3 "" H 8050 4250 50  0001 C CNN
 	1    8050 4250
@@
 F 0 "R31" V 10000 3900 50  0000 C CNN
 F 1 "33" V 10050 4150 50  0000 C CNN
-F 2 "" V 9980 4150 50  0001 C CNN
+F 2 "azonenberg_pcb:EIA_0402_RES_NOSILK" V 9980 4150 50  0001 C CNN
 F 3 "" H 10050 4150 50  0001 C CNN
 	1    10050 4150
@@
 F 0 "R32" V 10000 4100 50  0000 C CNN
 F 1 "33" V 10050 4350 50  0000 C CNN
-F 2 "" V 9980 4350 50  0001 C CNN
+F 2 "azonenberg_pcb:EIA_0402_RES_NOSILK" V 9980 4350 50  0001 C CNN
 F 3 "" H 10050 4350 50  0001 C CNN
 	1    10050 4350
@@
 F 0 "R27" V 7000 1000 50  0000 C CNN
 F 1 "33" V 7050 1250 50  0000 C CNN
-F 2 "" V 6980 1250 50  0001 C CNN
+F 2 "azonenberg_pcb:EIA_0402_RES_NOSILK" V 6980 1250 50  0001 C CNN
 F 3 "" H 7050 1250 50  0001 C CNN
 	1    7050 1250
@@
 F 0 "R26" V 4950 2150 50  0000 C CNN
 F 1 "33" V 5000 1950 50  0000 C CNN
-F 2 "" V 4930 1950 50  0001 C CNN
+F 2 "azonenberg_pcb:EIA_0402_RES_NOSILK" V 4930 1950 50  0001 C CNN
 F 3 "" H 5000 1950 50  0001 C CNN
 	1    5000 1950
@@
 F 0 "R28" V 7050 550 50  0000 C CNN
 F 1 "4.7K" V 7100 800 50  0000 C CNN
-F 2 "" V 7030 800 50  0001 C CNN
+F 2 "azonenberg_pcb:EIA_0402_RES_NOSILK" V 7030 800 50  0001 C CNN
 F 3 "" H 7100 800 50  0001 C CNN
 	1    7100 800
@@
 F 0 "R25" V 4650 2800 50  0000 C CNN
 F 1 "4.7K" V 4700 2600 50  0000 C CNN
-F 2 "" V 4630 2600 50  0001 C CNN
+F 2 "azonenberg_pcb:EIA_0402_RES_NOSILK" V 4630 2600 50  0001 C CNN
 F 3 "" H 4700 2600 50  0001 C CNN
 	1    4700 2600

Commit message: Added footprints for most ICs other than DC-DC modules
Parts:
- U29: footprint (none) -> azonenberg_pcb:DFN_8_1.27MM_6x5MM
- U4: footprint (none) -> azonenberg_pcb:BGA_196_15x15_FULLARRAY_1MM_FTGB196
Changed lines of the file:
@@
 F 0 "U4" H 2350 11475 50  0000 C CNN
 F 1 "XC7S6-1FTGB196C" H 2350 11384 50  0000 C CNN
-F 2 "" H 1600 6100 50  0001 C CNN
+F 2 "azonenberg_pcb:BGA_196_15x15_FULLARRAY_1MM_FTGB196" H 1600 6100 50  0001 C CNN
 F 3 "" H 1600 6100 50  0001 C CNN
 	1    1600 6100
@@
 F 0 "U4" H 6075 5075 50  0000 C CNN
 F 1 "XC7S6-1FTGB196C" H 6075 4984 50  0000 C CNN
-F 2 "" H 5600 2900 50  0001 C CNN
+F 2 "azonenberg_pcb:BGA_196_15x15_FULLARRAY_1MM_FTGB196" H 5600 2900 50  0001 C CNN
 F 3 "" H 5600 2900 50  0001 C CNN
 	2    5600 2900
@@
 F 0 "U29" H 8950 5137 60  0000 C CNN
 F 1 "S25FL128LAGNFV010" H 8950 5031 60  0000 C CNN
-F 2 "" H 8950 4450 60  0001 C CNN
+F 2 "azonenberg_pcb:DFN_8_1.27MM_6x5MM" H 8950 4450 60  0001 C CNN
 F 3 "" H 8950 4450 60  0000 C CNN
 	1    8950 4450

Commit message: Continued schematic review
Parts:
- added R248, R249, R250: 4.7K, azonenberg_pcb:EIA_0402_RES_NOSILK, symbol device:R
Connections:
- net 3V3: now also R248.1, R249.1, R250.1
- net S7_QSPI_CS_N: now also R248.2
- net S7_QSPI_DQ2: now also R249.2
- net S7_QSPI_DQ3: now also R250.2
Changed lines of the file:
@@
 Sheet 9 18
 Title "MAXWELL Main Board"
-Date "2020-06-24"
+Date "2020-06-25"
 Rev "0.1"
 Comp "Antikernel Labs"
@@
 	5100 2450 5400 2450
 NoConn ~ 2450 7550
+$Comp
+L device:R R248
+U 1 1 62C79BAD
+P 8050 3200
+F 0 "R248" V 8000 2950 50  0000 C CNN
+F 1 "4.7K" V 8050 3200 50  0000 C CNN
+F 2 "azonenberg_pcb:EIA_0402_RES_NOSILK" V 7980 3200 50  0001 C CNN
+F 3 "" H 8050 3200 50  0001 C CNN
+	1    8050 3200
+	0    1    1    0
+$EndComp
+Text Label 7650 3200 2    50   ~ 0
+S7_QSPI_CS_N
+Wire Wire Line
+	7650 3200 7900 3200
+$Comp
+L device:R R249
+U 1 1 62C7F795
+P 8050 3300
+F 0 "R249" V 8000 3050 50  0000 C CNN
+F 1 "4.7K" V 8050 3300 50  0000 C CNN
+F 2 "azonenberg_pcb:EIA_0402_RES_NOSILK" V 7980 3300 50  0001 C CNN
+F 3 "" H 8050 3300 50  0001 C CNN
+	1    8050 3300
+	0    1    1    0
+$EndComp
+Text Label 7650 3300 2    50   ~ 0
+S7_QSPI_DQ2
+Wire Wire Line
+	7650 3300 7900 3300
+$Comp
+L device:R R250
+U 1 1 62C85809
+P 8050 3400
+F 0 "R250" V 8000 3150 50  0000 C CNN
+F 1 "4.7K" V 8050 3400 50  0000 C CNN
+F 2 "azonenberg_pcb:EIA_0402_RES_NOSILK" V 7980 3400 50  0001 C CNN
+F 3 "" H 8050 3400 50  0001 C CNN
+	1    8050 3400
+	0    1    1    0
+$EndComp
+Text Label 7650 3400 2    50   ~ 0
+S7_QSPI_DQ3
+Wire Wire Line
+	7650 3400 7900 3400
+Text Label 8200 3200 0    50   ~ 0
+3V3
+Wire Wire Line
+	8200 3200 8200 3300
+Connection ~ 8200 3300
+Wire Wire Line
+	8200 3300 8200 3400
 $EndSCHEMATC

Commit message: Finished design review!!
Parts:
- added TP11, TP12, TP13, TP14: TESTPAD, azonenberg_pcb:TESTPOINT_SMT_0.5MM, symbol Connector:Conn_01x01
Connections:
- net GND: now also TP11.1 (Pin_1)
- net S7_DONE: now also TP14.1 (Pin_1)
- net S7_INIT_B: now also TP13.1 (Pin_1)
- net S7_RST_N: now also TP12.1 (Pin_1)
Changed lines of the file:
@@
 Wire Wire Line
 	8200 3300 8200 3400
+$Comp
+L Connector:Conn_01x01 TP11
+U 1 1 62EF70E0
+P 8750 1000
+F 0 "TP11" H 8668 775 50  0000 C CNN
+F 1 "TESTPAD" H 8668 866 50  0000 C CNN
+F 2 "azonenberg_pcb:TESTPOINT_SMT_0.5MM" H 8750 1000 50  0001 C CNN
+F 3 "~" H 8750 1000 50  0001 C CNN
+	1    8750 1000
+	-1   0    0    1
+$EndComp
+Text Label 8950 1000 0    50   ~ 0
+GND
+$Comp
+L Connector:Conn_01x01 TP12
+U 1 1 62EF7BAE
+P 8750 1350
+F 0 "TP12" H 8668 1125 50  0000 C CNN
+F 1 "TESTPAD" H 8668 1216 50  0000 C CNN
+F 2 "azonenberg_pcb:TESTPOINT_SMT_0.5MM" H 8750 1350 50  0001 C CNN
+F 3 "~" H 8750 1350 50  0001 C CNN
+	1    8750 1350
+	-1   0    0    1
+$EndComp
+Text Label 8950 1350 0    50   ~ 0
+S7_RST_N
+$Comp
+L Connector:Conn_01x01 TP13
+U 1 1 62EF8608
+P 8750 1700
+F 0 "TP13" H 8668 1475 50  0000 C CNN
+F 1 "TESTPAD" H 8668 1566 50  0000 C CNN
+F 2 "azonenberg_pcb:TESTPOINT_SMT_0.5MM" H 8750 1700 50  0001 C CNN
+F 3 "~" H 8750 1700 50  0001 C CNN
+	1    8750 1700
+	-1   0    0    1
+$EndComp
+Text Label 8950 1700 0    50   ~ 0
+S7_INIT_B
+$Comp
+L Connector:Conn_01x01 TP14
+U 1 1 62EF891B
+P 8750 2050
+F 0 "TP14" H 8668 1825 50  0000 C CNN
+F 1 "TESTPAD" H 8668 1916 50  0000 C CNN
+F 2 "azonenberg_pcb:TESTPOINT_SMT_0.5MM" H 8750 2050 50  0001 C CNN
+F 3 "~" H 8750 2050 50  0001 C CNN
+	1    8750 2050
+	-1   0    0    1
+$EndComp
+Text Label 8950 2050 0    50   ~ 0
+S7_DONE
 $EndSCHEMATC
