File: boards/probes/resistive-probe/resistive-probe.sch (KiCad schematic (older format))
At the start: 4 parts, among them P1 MMCX, P2 SOLDERPAD, P3 SOLDERPAD

Commit message: v0.3 AKL-PT2 layout
Parts:
- removed P1: MMCX, azonenberg_pcb:CONN_MMCX_LINX_CONNMMCX002SMD, symbol BNC
- removed P2, P3: SOLDERPAD, azonenberg_pcb:FLEX_SOLDERPAD, symbol CONN_01X01
- removed R1: R, azonenberg_pcb:EIA_0402_RES_NOSILK, symbol R
- added J1: SMA, azonenberg_pcb:CONN_SMA_EDGE_AMPHENOL_901_10511_3, symbol Connector:Conn_Coaxial
- added J2: TIP, azonenberg_pcb:TESTPOINT_BARETRACE_150UM, symbol Connector:Conn_01x01
- added J3: GND, azonenberg_pcb:TESTPOINT_BARETRACE_150UM, symbol Connector:Conn_01x01
- added R1: 50, azonenberg_pcb:EIA_0402_RES_NOSILK_FLIPCHIP, symbol device:R
- added R2, R3: 200, azonenberg_pcb:EIA_0402_RES_NOSILK_FLIPCHIP, symbol device:R
Connections:
- wire segments 4 -> 5
Other:
- note added: "All resistors Vishay FC0402 series\nFlip chip with no wraparound terminals"
- note removed: "R = 953 ohm + 49 in host provides 20.45x attenuation\nR= 0 ohm provides no attenuation"
Changed lines of the file:
@@
-EESchema Schematic File Version 2
-LIBS:analog-azonenberg
-LIBS:cmos
-LIBS:cypress-azonenberg
-LIBS:hirose-azonenberg
-LIBS:memory-azonenberg
-LIBS:microchip-azonenberg
-LIBS:osc-azonenberg
-LIBS:passive-azonenberg
-LIBS:power-azonenberg
-LIBS:special-azonenberg
-LIBS:xilinx-azonenberg
-LIBS:conn
-LIBS:device
+EESchema Schematic File Version 4
 LIBS:resistive-probe-cache
-EELAYER 26 0
+EELAYER 30 0
 EELAYER END
 $Descr A4 11693 8268
 encoding utf-8
 Sheet 1 1
-Title "STARSHIPRAIDER Resistive Probe"
-Date "2017-05-27"
-Rev "0.1"
+Title "AKL-PT2"
+Date "2020-10-02"
+Rev "0.3"
 Comp "Andrew Zonenberg"
 Comment1 ""
@@
 $EndDescr
 $Comp
-L CONN_01X01 P2
-U 1 1 5929E172
-P 7750 2750
-F 0 "P2" H 7828 2791 50  0000 L CNN
-F 1 "SOLDERPAD" H 7828 2700 50  0000 L CNN
-F 2 "azonenberg_pcb:FLEX_SOLDERPAD" H 7750 2750 50  0001 C CNN
-F 3 "" H 7750 2750 50  0000 C CNN
-	1    7750 2750
+L Connector:Conn_01x01 J2
+U 1 1 5F77A650
+P 6100 2900
+F 0 "J2" H 6180 2942 50  0000 L CNN
+F 1 "TIP" H 6180 2851 50  0000 L CNN
+F 2 "azonenberg_pcb:TESTPOINT_BARETRACE_150UM" H 6100 2900 50  0001 C CNN
+F 3 "~" H 6100 2900 50  0001 C CNN
+	1    6100 2900
 	1    0    0    -1
 $EndComp
 $Comp
-L CONN_01X01 P3
-U 1 1 5929E1F3
-P 7750 3100
-F 0 "P3" H 7828 3141 50  0000 L CNN
-F 1 "SOLDERPAD" H 7828 3050 50  0000 L CNN
-F 2 "azonenberg_pcb:FLEX_SOLDERPAD" H 7750 3100 50  0001 C CNN
-F 3 "" H 7750 3100 50  0000 C CNN
-	1    7750 3100
+L Connector:Conn_01x01 J3
+U 1 1 5F77A89F
+P 6100 3100
+F 0 "J3" H 6180 3142 50  0000 L CNN
+F 1 "GND" H 6180 3051 50  0000 L CNN
+F 2 "azonenberg_pcb:TESTPOINT_BARETRACE_150UM" H 6100 3100 50  0001 C CNN
+F 3 "~" H 6100 3100 50  0001 C CNN
+	1    6100 3100
 	1    0    0    -1
 $EndComp
-Text Label 7200 3100 2    60   ~ 0
-GND
-Wire Wire Line
-	6250 3100 7550 3100
 $Comp
-L R R1
-U 1 1 5929E268
-P 7200 2750
-F 0 "R1" V 7100 2750 50  0000 C CNN
-F 1 "R" V 7200 2750 50  0000 C CNN
-F 2 "azonenberg_pcb:EIA_0402_RES_NOSILK" V 7130 2750 50  0001 C CNN
-F 3 "" H 7200 2750 50  0000 C CNN
-	1    7200 2750
+L Connector:Conn_Coaxial J1
+U 1 1 5F77AC4B
+P 4250 2900
+F 0 "J1" H 4203 3138 50  0000 C CNN
+F 1 "SMA" H 4203 3047 50  0000 C CNN
+F 2 "azonenberg_pcb:CONN_SMA_EDGE_AMPHENOL_901_10511_3" H 4250 2900 50  0001 C CNN
+F 3 "" H 4250 2900 50  0001 C CNN
+	1    4250 2900
+	-1   0    0    -1
+$EndComp
+$Comp
+L device:R R3
+U 1 1 5F77B938
+P 5650 2900
+F 0 "R3" V 5443 2900 50  0000 C CNN
+F 1 "200" V 5534 2900 50  0000 C CNN
+F 2 "azonenberg_pcb:EIA_0402_RES_NOSILK_FLIPCHIP" V 5580 2900 50  0001 C CNN
+F 3 "" H 5650 2900 50  0001 C CNN
+	1    5650 2900
+	0    1    1    0
+$EndComp
+$Comp
+L device:R R2
+U 1 1 5F77BEDC
+P 5250 2900
+F 0 "R2" V 5043 2900 50  0000 C CNN
+F 1 "200" V 5134 2900 50  0000 C CNN
+F 2 "azonenberg_pcb:EIA_0402_RES_NOSILK_FLIPCHIP" V 5180 2900 50  0001 C CNN
+F 3 "" H 5250 2900 50  0001 C CNN
+	1    5250 2900
+	0    1    1    0
+$EndComp
+$Comp
+L device:R R1
+U 1 1 5F77C24C
+P 4850 2900
+F 0 "R1" V 4643 2900 50  0000 C CNN
+F 1 "50" V 4734 2900 50  0000 C CNN
+F 2 "azonenberg_pcb:EIA_0402_RES_NOSILK_FLIPCHIP" V 4780 2900 50  0001 C CNN
+F 3 "" H 4850 2900 50  0001 C CNN
+	1    4850 2900
 	0    1    1    0
 $EndComp
 Wire Wire Line
-	7350 2750 7550 2750
-Text Notes 7100 2550 0    60   ~ 0
-R = 953 ohm + 49 in host provides 20.45x attenuation\nR= 0 ohm provides no attenuation
-$Comp
-L BNC P1
-U 1 1 5929E35B
-P 6250 2750
-F 0 "P1" H 6351 2726 50  0000 L CNN
-F 1 "MMCX" H 6351 2635 50  0000 L CNN
-F 2 "azonenberg_pcb:CONN_MMCX_LINX_CONNMMCX002SMD" H 6250 2750 50  0001 C CNN
-F 3 "" H 6250 2750 50  0000 C CNN
-	1    6250 2750
-	-1   0    0    -1
-$EndComp
+	4400 2900 4700 2900
 Wire Wire Line
-	6400 2750 7050 2750
+	5000 2900 5100 2900
 Wire Wire Line
-	6250 3100 6250 2950
+	5900 3100 4250 3100
+Wire Wire Line
+	5400 2900 5500 2900
+Wire Wire Line
+	5800 2900 5900 2900
+Text Notes 4750 2600 0    50   ~ 0
+All resistors Vishay FC0402 series\nFlip chip with no wraparound terminals
+Text Label 5650 3100 0    50   ~ 0
+GND
 $EndSCHEMATC
