File: boards/probes/akl-pt2/akl-pt2.kicad_pcb (KiCad board)
At the start: 2 copper layers, 150.5 x 8 mm, 6 parts, among them J1 SMA, J2 TIP, J3 GND

Commit message: Finished AKL-PT2 layout changes for v0.4
Routing:
- net Net-(J2-Pad1): track 0.93 -> 1.68 mm, vias 0 -> 2
- net /GND: track 284.6 -> 285.3 mm, vias 284 -> 286
Other:
- outline, holes or cut-outs redrawn
- board text added: "AKL-PT2 / A. Zonenberg / Antikernel Labs / Symbiotic EDA / v0.4 / 2020-11-26"
- board text removed: "AKL-PT2 / A. Zonenberg / Antikernel Labs / Symbiotic EDA / v0.3 / 2020-10-04"
Changed lines of the file:
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@@
     (thickness 0.23)
     (drawings 15)
-    (tracks 575)
+    (tracks 583)
     (zones 0)
     (modules 6)
@@
   )
   (setup
-    (last_trace_width 0.2)
+    (last_trace_width 0.125)
     (user_trace_width 0.2)
     (user_trace_width 0.225)
     (trace_clearance 0.125)
-    (zone_clearance 0.2)
+    (zone_clearance 0.225)
     (zone_45_only no)
     (trace_min 0.125)
@@
       (rotate (xyz 90 0 0))
     )
-    (model /nfs4/home/azonenberg/code/starshipraider/mechanical/resistive-probe/tube.step
-      (offset (xyz 6 0 0))
-      (scale (xyz 1 1 1))
-      (rotate (xyz 90 0 90))
-    )
   )
   (gr_arc (start 94.75 54) (end 94.75 54.25) (angle -90) (layer Edge.Cuts) (width 0.05))
   (gr_arc (start 94.75 46.5) (end 95 46.5) (angle -90) (layer Edge.Cuts) (width 0.05))
   (gr_arc (start 95.25 52) (end 95.25 51.75) (angle -90) (layer Edge.Cuts) (width 0.05))
-  (gr_arc (start 95.25 48.25) (end 95 48.25) (angle -90) (layer Edge.Cuts) (width 0.05))
+  (gr_arc (start 95.25 48.5) (end 95 48.5) (angle -90) (layer Edge.Cuts) (width 0.05))
   (gr_line (start 236.75 51.75) (end 95.25 51.75) (layer Edge.Cuts) (width 0.05))
   (gr_arc (start 236.75 51.5) (end 236.75 51.75) (angle -90) (layer Edge.Cuts) (width 0.05))
   (gr_line (start 237 49) (end 237 51.5) (layer Edge.Cuts) (width 0.05))
   (gr_arc (start 236.75 49) (end 237 49) (angle -90) (layer Edge.Cuts) (width 0.05))
-  (gr_line (start 95.25 48.5) (end 236.75 48.75) (layer Edge.Cuts) (width 0.05))
-  (gr_text "AKL-PT2 / A. Zonenberg / Antikernel Labs / Symbiotic EDA / v0.3 / 2020-10-04" (at 127 50.25) (layer B.SilkS)
+  (gr_line (start 95.25 48.75) (end 236.75 48.75) (layer Edge.Cuts) (width 0.05))
+  (gr_text "AKL-PT2 / A. Zonenberg / Antikernel Labs / Symbiotic EDA / v0.4 / 2020-11-26" (at 127 50.25) (layer B.SilkS)
     (effects (font (size 1 1) (thickness 0.15)) (justify mirror))
   )
@@
   (gr_line (start 86.5 46.25) (end 86.5 54.25) (layer Edge.Cuts) (width 0.05))
   (gr_line (start 94.75 46.25) (end 86.5 46.25) (layer Edge.Cuts) (width 0.05))
-  (gr_line (start 95 48.25) (end 95 46.5) (layer Edge.Cuts) (width 0.05))
+  (gr_line (start 95 48.5) (end 95 46.5) (layer Edge.Cuts) (width 0.05))
   (via (at 235.5 51) (size 0.55) (drill 0.25) (layers F.Cu B.Cu) (net 1))
   (segment (start 236.45 50.75) (end 235.75 50.75) (width 0.2) (layer F.Cu) (net 1))
@@
   (via (at 92.5 49.5) (size 0.55) (drill 0.25) (layers F.Cu B.Cu) (net 1))
   (segment (start 93.5 49.5) (end 92.5 49.5) (width 0.225) (layer B.Cu) (net 1))
-  (segment (start 231.9 49.95) (end 231.6 50.25) (width 0.225) (layer F.Cu) (net 2))
-  (segment (start 232.4 49.95) (end 231.9 49.95) (width 0.225) (layer F.Cu) (net 2))
-  (segment (start 92.4 50.25) (end 89.35 50.25) (width 0.225) (layer F.Cu) (net 2))
-  (segment (start 231.6 50.25) (end 92.4 50.25) (width 0.225) (layer F.Cu) (net 2))
+  (via (at 236.25 50.75) (size 0.55) (drill 0.25) (layers F.Cu B.Cu) (net 1))
+  (segment (start 236.45 50.75) (end 236.25 50.75) (width 0.125) (layer F.Cu) (net 1))
+  (via (at 236.95 50.75) (size 0.55) (drill 0.25) (layers F.Cu B.Cu) (net 1))
+  (segment (start 236.45 50.75) (end 237 50.75) (width 0.125) (layer F.Cu) (net 1))
+  (segment (start 231.9 49.95) (end 231.6 50.25) (width 0.2) (layer F.Cu) (net 2))
+  (segment (start 232.4 49.95) (end 231.9 49.95) (width 0.2) (layer F.Cu) (net 2))
+  (segment (start 92.4 50.25) (end 89.35 50.25) (width 0.2) (layer F.Cu) (net 2))
+  (segment (start 231.6 50.25) (end 92.4 50.25) (width 0.2) (layer F.Cu) (net 2))
   (segment (start 235.8 49.75) (end 235.6 49.95) (width 0.225) (layer F.Cu) (net 3))
   (segment (start 236.45 49.75) (end 235.8 49.75) (width 0.2) (layer F.Cu) (net 3))
-  (zone (net 0) (net_name "") (layer F.Mask) (hatch edge 0.508)
-    (connect_pads (clearance 0.2))
-    (min_thickness 0.254)
-    (fill yes (arc_segments 32) (thermal_gap 0.508) (thermal_bridge_width 0.508))
-    (polygon
-      (pts
-        (xy 232 49) (xy 232 51.5) (xy 92.5 51.5) (xy 92.5 49) (xy 111.5 49)
-      )
-    )
-  )
+  (via (at 236.25 49.75) (size 0.55) (drill 0.25) (layers F.Cu B.Cu) (net 3))
+  (segment (start 236.45 49.75) (end 236.25 49.75) (width 0.125) (layer F.Cu) (net 3))
+  (via (at 236.95 49.75) (size 0.55) (drill 0.25) (layers F.Cu B.Cu) (net 3))
+  (segment (start 236.45 49.75) (end 237 49.75) (width 0.125) (layer F.Cu) (net 3))
   (zone (net 1) (net_name /GND) (layer B.Cu) (hatch edge 0.508)
     (connect_pads (clearance 0.1))
@@
   )
   (zone (net 1) (net_name /GND) (layer F.Cu) (hatch edge 0.508)
-    (connect_pads yes (clearance 0.2))
+    (connect_pads yes (clearance 0.225))
     (min_thickness 0.1)
     (fill yes (arc_segments 32) (thermal_gap 0.1) (thermal_bridge_width 0.125))
@@
       )
     )
+  )
+  (zone (net 0) (net_name "") (layer F.Mask) (hatch edge 0.508)
+    (connect_pads yes (clearance 0.225))
+    (min_thickness 0.1)
+    (fill yes (arc_segments 32) (thermal_gap 0.1) (thermal_bridge_width 0.125))
+    (polygon
+      (pts
+        (xy 86.5 49.35) (xy 86.5 51.225) (xy 92.2 51.225) (xy 92.2 49.35)
+      )
+    )

Commit message: Initial board design for AKL-PT2 v0.5
Other:
- board text added: "AKL-PT2 / A. Zonenberg / Antikernel Labs / Symbiotic EDA / v0.5 / 2020-12-22"
- board text added: "FR4 stiffener 1.4 mm nominal Total thickness of stiffener and PCB not to exceed 1.6 mm"
- board text added: "Polyimide stiffener 0.2mm thick"
- board text removed: "AKL-PT2 / A. Zonenberg / Antikernel Labs / Symbiotic EDA / v0.4 / 2020-11-26"
Changed lines of the file:
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@@
   (general
     (thickness 0.23)
-    (drawings 15)
+    (drawings 25)
     (tracks 583)
     (zones 0)
@@
     (39 F.Mask user)
     (40 Dwgs.User user)
+    (42 Eco1.User user)
+    (43 Eco2.User user)
     (44 Edge.Cuts user)
     (45 Margin user)
@@
     (visible_elements FFFFFF7F)
     (pcbplotparams
-      (layerselection 0x030f8_ffffffff)
+      (layerselection 0x03cf8_ffffffff)
       (usegerberextensions false)
       (usegerberattributes true)
@@
     )
   )
+  (gr_text "Polyimide stiffener\n0.2mm thick" (at 233.7 47) (layer Eco2.User)
+    (effects (font (size 1 1) (thickness 0.05)))
+  )
+  (gr_line (start 235.9 48.8) (end 230.5 48.8) (layer Eco2.User) (width 0.05))
+  (gr_line (start 235.9 51.7) (end 235.9 48.8) (layer Eco2.User) (width 0.05))
+  (gr_line (start 230.5 51.7) (end 235.9 51.7) (layer Eco2.User) (width 0.05))
+  (gr_line (start 230.5 48.8) (end 230.5 51.7) (layer Eco2.User) (width 0.05))
+  (gr_text "FR4 stiffener 1.4 mm nominal\nTotal thickness of stiffener and\nPCB not to exceed 1.6 mm" (at 91.5 44.1) (layer Eco1.User)
+    (effects (font (size 0.75 0.75) (thickness 0.05)))
+  )
+  (gr_line (start 94 46.5) (end 86.5 46.5) (layer Eco1.User) (width 0.05))
+  (gr_line (start 94 54) (end 94 46.5) (layer Eco1.User) (width 0.05))
+  (gr_line (start 86.5 54) (end 94 54) (layer Eco1.User) (width 0.05))
+  (gr_line (start 86.5 46.5) (end 86.5 54) (layer Eco1.User) (width 0.05))
   (gr_arc (start 94.75 54) (end 94.75 54.25) (angle -90) (layer Edge.Cuts) (width 0.05))
   (gr_arc (start 94.75 46.5) (end 95 46.5) (angle -90) (layer Edge.Cuts) (width 0.05))
@@
   (gr_arc (start 236.75 49) (end 237 49) (angle -90) (layer Edge.Cuts) (width 0.05))
   (gr_line (start 95.25 48.75) (end 236.75 48.75) (layer Edge.Cuts) (width 0.05))
-  (gr_text "AKL-PT2 / A. Zonenberg / Antikernel Labs / Symbiotic EDA / v0.4 / 2020-11-26" (at 127 50.25) (layer B.SilkS)
+  (gr_text "AKL-PT2 / A. Zonenberg / Antikernel Labs / Symbiotic EDA / v0.5 / 2020-12-22" (at 127 50.25) (layer B.SilkS)
     (effects (font (size 1 1) (thickness 0.15)) (justify mirror))
   )
@@
       )
     )
+  )
+  (zone (net 0) (net_name "") (layer F.Mask) (hatch edge 0.508)
+    (connect_pads (clearance 0.225))
+    (min_thickness 0.254)
+    (fill yes (arc_segments 32) (thermal_gap 0.508) (thermal_bridge_width 0.508))
+    (polygon
+      (pts
+        (xy 235.9 49.3) (xy 235.9 51.2) (xy 237 51.2) (xy 237 49.3)
+      )
+    )
+  )
+  (zone (net 0) (net_name "") (layer B.Mask) (hatch edge 0.508)
+    (connect_pads (clearance 0.225))
+    (min_thickness 0.254)
+    (fill yes (arc_segments 32) (thermal_gap 0.508) (thermal_bridge_width 0.508))
+    (polygon
+      (pts
+        (xy 236.6 49.3) (xy 236.6 51.2) (xy 237 51.2) (xy 237 49.3)
+      )
+    )
